Commit message: lp:844934 lp:850726 lp:844723 working on the gazebo model.

File: model/robots/xacro/arm_and_hand_muscle.urdf.xacro (robot description, xacro)
@@ -6,8 +6,13 @@
   <include filename="$(find sr_hand)/model/desk/desk.urdf.xacro" />
   <xacro:desk/>
-  <joint name="base_fix" type="fixed">
+  <joint name="arm_to_desk_fixed" type="fixed">
     <parent link="desk_pillar"/>
     <child link="shadowarm_base"/>
     <origin rpy="0 0 0" xyz="0 0 1.0"/>
+  </joint>
+  <joint name="base_fix" type="fixed">
+    <parent link="world"/>
+    <child link="desk_support"/>
+    <origin rpy="0 0 0" xyz="0 0 0"/>
   </joint>
   <xacro:sr_arm_muscle>

File: model/robots/xacro/sr_arm_motor.urdf.xacro (robot description, xacro)
@@ -4,7 +4,19 @@
        xmlns:xacro="http://www.ros.org/wiki/xacro"
        name="sr_arm_motor">
+  <include filename="$(find sr_hand)/model/desk/desk.urdf.xacro" />
   <include filename="$(find sr_hand)/model/materials.urdf.xacro" />
   <include filename="$(find sr_hand)/model/arm_urdf/full_arm_motor.urdf.xacro" />
   <include filename="$(find sr_hand)/model/gazebo/gazebo.urdf.xacro" />
+  <xacro:desk/>
+  <joint name="arm_to_desk_fixed" type="fixed">
+    <parent link="desk_pillar"/>
+    <child link="shadowarm_base"/>
+    <origin rpy="0 0 0" xyz="0 0 1.0"/>
+  </joint>
+  <joint name="base_fix" type="fixed">
+    <parent link="world"/>
+    <child link="desk_support"/>
+    <origin rpy="0 0 0" xyz="0 0 0"/>
+  </joint>
   <xacro:sr_arm_motor>
   </xacro:sr_arm_motor>
