Commit message: added desk to muscle arm

File: model/robots/xacro/sr_arm_muscle.urdf.xacro (robot description, xacro)
@@ -4,7 +4,19 @@
        xmlns:xacro="http://www.ros.org/wiki/xacro"
        name="sr_arm_muscle">
+  <include filename="$(find sr_hand)/model/desk/desk.urdf.xacro" />
   <include filename="$(find sr_hand)/model/materials.urdf.xacro" />
   <include filename="$(find sr_hand)/model/arm_urdf/full_arm_muscle.urdf.xacro" />
   <include filename="$(find sr_hand)/model/gazebo/gazebo.urdf.xacro" />
+  <xacro:desk/>
+  <joint name="arm_to_desk_fixed" type="fixed">
+    <parent link="desk_pillar"/>
+    <child link="shadowarm_base"/>
+    <origin rpy="0 0 0" xyz="0 0 1.0"/>
+  </joint>
+  <joint name="base_fix" type="fixed">
+    <parent link="world"/>
+    <child link="desk_support"/>
+    <origin rpy="0 0 0" xyz="0 0 0"/>
+  </joint>
   <xacro:sr_arm_muscle>
   </xacro:sr_arm_muscle>
