Commit message: commiting the generated models to help debugging.

File: model/robots/arm_and_hand_motor.urdf (robot description, URDF)
Before this commit: robot arm_and_hand, 31 links, 30 joints
Links:
- added link desk_pillar, mass 100.0; collision cylinder length=1.0 radius=0.1; visual cylinder length=1.0 radius=0.1
- added link desk_support, mass 1000.0; collision cylinder length=0.02 radius=1.0; visual cylinder length=0.02 radius=1.0
Joints:
- added joint arm_to_desk_fixed: type fixed, parent desk_pillar, child shadowarm_base, origin xyz=0 0 1.0 rpy=0 0 0
- added joint desk_joint: type fixed, parent desk_support, child desk_pillar, origin xyz=0 0 0.01 rpy=0 0 0
- joint arm_link: origin xyz=0 0 0 rpy=1.57079632679 0 1.57079632679 -> xyz=0 0 0 rpy=0 0 3.14159265359
- joint base_fix: child shadowarm_base -> desk_support

File: model/robots/arm_and_hand_muscle.urdf (robot description, URDF)
Before this commit: robot arm_and_hand, 31 links, 30 joints
Links:
- added link desk_pillar, mass 100.0; collision cylinder length=1.0 radius=0.1; visual cylinder length=1.0 radius=0.1
- added link desk_support, mass 1000.0; collision cylinder length=0.02 radius=1.0; visual cylinder length=0.02 radius=1.0
Joints:
- added joint arm_to_desk_fixed: type fixed, parent desk_pillar, child shadowarm_base, origin xyz=0 0 1.0 rpy=0 0 0
- added joint desk_joint: type fixed, parent desk_support, child desk_pillar, origin xyz=0 0 0.01 rpy=0 0 0
- joint arm_link: origin xyz=0 0 0 rpy=1.57079632679 0 1.57079632679 -> xyz=0 0 0 rpy=0 0 3.14159265359
- joint base_fix: child shadowarm_base -> desk_support

File: model/robots/sr_arm_motor.urdf (robot description, URDF)
Before this commit: robot sr_arm_motor, 6 links, 5 joints
Links:
- added link desk_pillar, mass 100.0; collision cylinder length=1.0 radius=0.1; visual cylinder length=1.0 radius=0.1
- added link desk_support, mass 1000.0; collision cylinder length=0.02 radius=1.0; visual cylinder length=0.02 radius=1.0
Joints:
- added joint arm_to_desk_fixed: type fixed, parent desk_pillar, child shadowarm_base, origin xyz=0 0 1.0 rpy=0 0 0
- added joint desk_joint: type fixed, parent desk_support, child desk_pillar, origin xyz=0 0 0.01 rpy=0 0 0
- joint base_fix: child shadowarm_base -> desk_support

File: model/robots/sr_arm_muscle.urdf (robot description, URDF)
Before this commit: robot sr_arm_muscle, 6 links, 5 joints
Links:
- added link desk_pillar, mass 100.0; collision cylinder length=1.0 radius=0.1; visual cylinder length=1.0 radius=0.1
- added link desk_support, mass 1000.0; collision cylinder length=0.02 radius=1.0; visual cylinder length=0.02 radius=1.0
Joints:
- added joint arm_to_desk_fixed: type fixed, parent desk_pillar, child shadowarm_base, origin xyz=0 0 1.0 rpy=0 0 0
- added joint desk_joint: type fixed, parent desk_support, child desk_pillar, origin xyz=0 0 0.01 rpy=0 0 0
- joint base_fix: child shadowarm_base -> desk_support
