Commit message: Added the long "palm" of the finger unit as a simple box.

File: model/hand_urdf/one_finger_unit_motor.urdf.xacro (robot description, xacro)
@@ -8,6 +8,33 @@
     <xacro:forearm_motor>
     </xacro:forearm_motor>
-    <xacro:finger link_prefix="mf" joint_prefix="MF" parent="forearm_motor">
-      <origin xyz="0.011 0 0.33" rpy="0 0 0" />
+    <link name="dummy_palm">
+      <inertial>
+	<mass value="0.010" />
+	<origin xyz="0 0 0" />
+	<inertia  ixx="1.0" ixy="0.0"  ixz="0.0"  iyy="0.0"  iyz="0.0"
+	izz="0.0" />
+      </inertial>
+      <visual>
+	<origin xyz="0 0 0.0505" rpy="0 0 0" />
+	<geometry name="dummy_palm_visual">
+	  <box size="0.015 0.015 0.110" />
+	</geometry>
+      <material name="Grey" />
+      </visual>
+      <collision>
+	<origin xyz="0 0 0.0" rpy="0 0 0" />
+	<geometry name="dummy_palm_collision_geom">
+	  <box size="0.015 0.015 0.110" />
+	</geometry>
+      </collision>
+    </link>
+    <joint name="forearm_to_dummy" type="fixed">
+      <parent link="forearm_motor"/>
+      <child link="dummy_palm"/>
+      <origin xyz="0.011 0.010 0.22" rpy="0 0 0"/>
+    </joint>
+    <!-- mfknuckle is at [0.011 -0.01 0.346] from the bottom of forearm_motor -->
+    <xacro:finger link_prefix="mf" joint_prefix="MF" parent="dummy_palm">
+      <origin xyz="0.0 0 0.116" rpy="0 0 0" />
       <axis xyz="0 -1 0" />
     </xacro:finger>
