Commit message: Add thumb to left hand model.

File: model/hand_urdf/full_hand_left_motor.urdf.xacro (robot description, xacro)
@@ -33,8 +33,6 @@
     <xacro:little_finger_left link_prefix="lf" joint_prefix="LF" parent="palm">
     </xacro:little_finger_left>
-    <!--
-    <xacro:thumb parent="palm">
-    </xacro:thumb>
-    -->
+    <xacro:thumb_left parent="palm">
+    </xacro:thumb_left>
   </xacro:macro>
 </robot>

File: model/hand_urdf/thumb/thbase.urdf.xacro (robot description, xacro)
@@ -7,4 +7,5 @@
        xmlns:geom="http://playerstage.sourceforge.net/gazebo/xmlschema/#geom">
   <include filename="$(find sr_hand)/model/hand_urdf/thumb/thbase.transmission.xacro" />
+  <!-- Right Hand -->
   <xacro:macro name="thbase" params="parent">
     <link name="thbase">
@@ -56,3 +57,53 @@
     <xacro:thbase_transmission />
   </xacro:macro>
+  <!-- Left Hand -->
+  <xacro:macro name="thbase_left" params="parent">
+    <link name="thbase">
+      <inertial>
+	<mass value="0.010" />
+	<origin xyz="-0.034 0.0085 0.029" rpy="0 0 0"/>
+	<inertia  ixx="0.0" ixy="0.0"  ixz="0.0"  iyy="0.0"  iyz="0.0"
+	izz="0.1" />
+      </inertial>
+      <visual>
+	<origin xyz="0 0 0" rpy="0 0 0" />
+	<geometry name="thbase_visual">
+	  <box size="0.001 0.001 0.001" />
+	</geometry>
+      <material name="shadow_thbase_material">
+	  <color rgba="0.5 0.5 0.5 1.0"/>
+	</material>
+      </visual>
+      <collision>
+	<origin xyz="0 0 0" rpy="0 0 0 " />
+	<geometry name="thbase_collision_geom">
+	  <box size="0.001 0.001 0.001" />
+	</geometry>
+      </collision>
+    </link>
+    <gazebo reference="thbase">
+      <sensor:contact name="thbase_contact_sensor">
+        <geom>thbase_geom</geom>
+       <updateRate>100.0</updateRate>
+        <controller:gazebo_ros_bumper name="thbase_gazebo_ros_bumper_controller" plugin="libgazebo_ros_bumper.so">
+          <alwaysOn>true</alwaysOn>
+          <updateRate>100.0</updateRate>
+          <frameName>thbase</frameName>
+          <bumperTopicName>thbase_bumper</bumperTopicName>
+          <interface:bumper name="thbase_gazebo_ros_bumper_iface" />
+        </controller:gazebo_ros_bumper>
+      </sensor:contact>
+      <material>Gazebo/Grey</material>
+    </gazebo>
+    <joint name="THJ5" type="revolute">
+      <parent link="${parent}"/>
+      <child link="thbase"/>
+      <origin xyz="-0.034 -0.0085 0.029" rpy="0 ${M_PI/4} ${M_PI}" />
+      <axis xyz="0 0 1" />
+      <limit lower="-1.047" upper="1.047" effort="10"
+      velocity="1.0" />
+      <dynamics damping="50.5"/>
+    </joint>
+    <xacro:thbase_transmission />
+  </xacro:macro>
 </robot>

File: model/hand_urdf/thumb/thproximal.urdf.xacro (robot description, xacro)
@@ -7,5 +7,15 @@
        xmlns:geom="http://playerstage.sourceforge.net/gazebo/xmlschema/#geom">
   <include filename="$(find sr_hand)/model/hand_urdf/thumb/thproximal.transmission.xacro" />
+  <!-- Right Hand -->
   <xacro:macro name="thproximal" params="parent">
+      <xacro:thproximal_base parent="${parent}" reflect="1" />
+  </xacro:macro>
+  <!-- Left Hand -->
+  <xacro:macro name="thproximal_left" params="parent">
+      <xacro:thproximal_base parent="${parent}" reflect="-1" />
+  </xacro:macro>
+  <!-- Macro to used to generate left and right handed versions.
+  DO NOT use out side of here ie treat as a private macro -->
+  <xacro:macro name="thproximal_base" params="parent reflect">
     <link name="thproximal">
       <inertial>
@@ -48,5 +58,5 @@
       <child link="thproximal"/>
       <origin xyz="0 0 0" rpy="0 0 0" />
-      <axis xyz="1 0 0" />
+      <axis xyz="${reflect*1} 0 0" />
       <limit lower="0" upper="1.309" effort="10"
       velocity="1.0" />

File: model/hand_urdf/thumb/thumb.urdf.xacro (robot description, xacro)
@@ -5,4 +5,5 @@
   <include filename="$(find sr_hand)/model/hand_urdf/thumb/thmiddle.urdf.xacro" />
   <include filename="$(find sr_hand)/model/hand_urdf/thumb/thdistal.urdf.xacro" />
+  <!-- Right Hand -->
   <xacro:macro name="thumb" params="parent">
     <xacro:thbase parent="${parent}">
@@ -10,4 +11,17 @@
     <xacro:thproximal parent="thbase">
     </xacro:thproximal>
+    <xacro:thumb_common />
+  </xacro:macro>
+  <!-- Left Hand -->
+  <xacro:macro name="thumb_left" params="parent">
+    <xacro:thbase_left parent="${parent}">
+    </xacro:thbase_left>
+    <xacro:thproximal_left parent="thbase">
+    </xacro:thproximal_left>
+    <xacro:thumb_common />
+  </xacro:macro>
+  <!-- Macro for common parts in left and right handed versions.
+  DO NOT use out side of here ie treat as a private macro -->
+  <xacro:macro name="thumb_common">
     <xacro:thhub parent="thproximal">
     </xacro:thhub>

Commit message: Left hand version of wrist.
Used a mirrored mesh to easily make a left hand version of wrist.

Left hand model is now basically complete and seems to move ok under control
from sr_control_gui. Next just need to tidy up the palm and shadow hand files
to use the _left macro idion instead of copied files to get rid of the
duplication.

File: model/hand_urdf/full_hand_left_motor.urdf.xacro (robot description, xacro)
@@ -14,7 +14,7 @@
     <xacro:forearm_motor>
     </xacro:forearm_motor>
-    <xacro:wrist parent="forearm_motor">
+    <xacro:wrist_left parent="forearm_motor">
       <origin xyz="0 -0.010 0.213" rpy="0 0 0" />
-    </xacro:wrist>
+    </xacro:wrist_left>
     <xacro:palm parent="wrist">
     </xacro:palm>

File: model/hand_urdf/wrist/wrist.urdf.xacro (robot description, xacro)
@@ -1,5 +1,17 @@
 <robot xmlns:xacro="http://ros.org/wiki/xacro">
   <include filename="$(find sr_hand)/model/hand_urdf/wrist/wrist.transmission.xacro" />
+  <!-- Right Hand -->
   <xacro:macro name="wrist" params="parent *origin">
+    <xacro:wrist_base parent="${parent}" mesh="wrist.mesh">
+      <insert_block name="origin" />
+    </xacro:wrist_base>
+  </xacro:macro>
+  <!-- Left Hand -->
+  <xacro:macro name="wrist_left" params="parent *origin">
+    <xacro:wrist_base parent="${parent}" mesh="wrist_left.mesh">
+      <insert_block name="origin" />
+    </xacro:wrist_base>
+  </xacro:macro>
+  <xacro:macro name="wrist_base" params="parent *origin mesh">
     <link name="wrist" >
       <inertial>
@@ -12,5 +24,5 @@
 	<origin xyz="0 0 0" rpy="0 0 0" />
 	<geometry name="wrist_visual">
-	  <mesh filename="package://sr_hand/model/meshes/wrist.mesh" scale="0.001 0.001 0.001" />
+      <mesh filename="package://sr_hand/model/meshes/${mesh}" scale="0.001 0.001 0.001" />
 	</geometry>
 	<material name="LightGrey" />

Commit message: Remove commented out property, not going to use it anymore!

File: model/hand_urdf/full_hand_left_motor.urdf.xacro (robot description, xacro)
@@ -11,5 +11,4 @@
   <include filename="$(find sr_hand)/model/hand_urdf/thumb/thumb.urdf.xacro" />
   <xacro:macro name="shadowhand_motor">
-      <!-- <xacro:property name="reflect" value="-1" /> -->
     <xacro:forearm_motor>
     </xacro:forearm_motor>

Commit message: Remove seperate left hand palm file and replace with palm_left macro. Removes all the duplication.

File: model/hand_urdf/full_hand_left_motor.urdf.xacro (robot description, xacro)
@@ -5,6 +5,5 @@
   <include filename="$(find sr_hand)/model/hand_urdf/forearm/forearm_motor.urdf.xacro" />
   <include filename="$(find sr_hand)/model/hand_urdf/wrist/wrist.urdf.xacro" />
-  <!-- <include filename="$(find sr_hand)/model/hand_urdf/palm/palm.urdf.xacro" /> -->
-  <include filename="$(find sr_hand)/model/hand_urdf/palm/palm_left.urdf.xacro" />
+  <include filename="$(find sr_hand)/model/hand_urdf/palm/palm.urdf.xacro" />
   <include filename="$(find sr_hand)/model/hand_urdf/finger/classic_finger.urdf.xacro" />
   <include filename="$(find sr_hand)/model/hand_urdf/finger/little_finger.urdf.xacro" />
@@ -16,6 +15,6 @@
       <origin xyz="0 -0.010 0.213" rpy="0 0 0" />
     </xacro:wrist_left>
-    <xacro:palm parent="wrist">
-    </xacro:palm>
+    <xacro:palm_left parent="wrist">
+    </xacro:palm_left>
     <xacro:finger link_prefix="ff" joint_prefix="FF" parent="palm">
       <origin xyz="-0.033 0 0.095" rpy="0 0 0" />

File: model/hand_urdf/palm/palm.urdf.xacro (robot description, xacro)
@@ -7,5 +7,15 @@
        xmlns:geom="http://playerstage.sourceforge.net/gazebo/xmlschema/#geom">
   <include filename="$(find sr_hand)/model/hand_urdf/palm/palm.transmission.xacro" />
+  <!-- Right Hand -->
   <xacro:macro name="palm" params="parent">
+    <xacro:palm_base parent="${parent}" mesh="palm.mesh" />
+  </xacro:macro>
+  <!-- Left Hand -->
+  <xacro:macro name="palm_left" params="parent">
+    <xacro:palm_base parent="${parent}" mesh="palm_left.mesh" />
+  </xacro:macro>
+  <!-- Macro to used to generate left and right handed versions.
+  DO NOT use out side of here ie treat as a private macro -->
+  <xacro:macro name="palm_base" params="parent mesh">
     <link name="palm" >
       <inertial>
@@ -17,5 +27,5 @@
 	<origin xyz="0 0 0" rpy="0 0 0" />
 	<geometry name="palm_visual">
-	  <mesh filename="package://sr_hand/model/meshes/palm.mesh" scale="0.001 0.001 0.001" />
+      <mesh filename="package://sr_hand/model/meshes/${mesh}" scale="0.001 0.001 0.001" />
 	</geometry>
 	<material name="Grey"/>
