Commit message: Wrist is closer to the front than to the back in the motor hand!

File: model/hand_urdf/full_hand_motor.urdf.xacro (robot description, xacro)
@@ -13,5 +13,5 @@
     </xacro:forearm_motor>
     <xacro:wrist parent="forearm_motor">
-      <origin xyz="0 0.010 0.213" rpy="0 0 0" />
+      <origin xyz="0 0.010 0.213" rpy="0 0 3.14" />
     </xacro:wrist>
     <xacro:palm parent="wrist">

File: model/hand_urdf/one_finger_unit_motor.urdf.xacro (robot description, xacro)
@@ -32,5 +32,5 @@
       <parent link="forearm_motor"/>
       <child link="dummy_palm"/>
-      <origin xyz="0.011 0.010 0.22" rpy="0 0 0"/>
+      <origin xyz="0.011 0.010 0.22" rpy="0 0 3.14"/>
     </joint>
     <!-- mfknuckle is at [0.011 -0.01 0.346] from the bottom of forearm_motor -->

Commit message: Corrected sr_arm_motor_finger_ik.launch to use same syntax as sr_arm_motor.launch (this file requires some configs from sr-manipulation, which should be changed) Corrected urdf.xacro of wrist and palm + changed forearm mesh to comply with corrected wrist placement Changed arm_link to fixed instead of revolute (this fix is required for arm reverse kinematic to work) Corrected kinematics_tests to work with new transmission J0 in gazebo and in real world

File: model/hand_urdf/full_hand_motor.urdf.xacro (robot description, xacro)
@@ -13,5 +13,5 @@
     </xacro:forearm_motor>
     <xacro:wrist parent="forearm_motor">
-      <origin xyz="0 0.010 0.213" rpy="0 0 3.14" />
+      <origin xyz="0 -0.010 0.213" rpy="0 0 0" />
     </xacro:wrist>
     <xacro:palm parent="wrist">

File: model/hand_urdf/palm/palm.urdf.xacro (robot description, xacro)
@@ -10,5 +10,5 @@
     <link name="palm" >
       <inertial>
-	<origin xyz="0 0.010 0.247" rpy="0 0 0" />
+	<origin xyz="0 0 0.247" rpy="0 0 0" />
 	<mass value="0.3" />
 	<inertia  ixx="1.0" ixy="0.0"  ixz="0.0"  iyy="0.0"  iyz="0.0"

File: model/hand_urdf/wrist/wrist.urdf.xacro (robot description, xacro)
@@ -7,6 +7,5 @@
 	<insert_block name="origin" />
 	<mass value="0.3" />
-	<inertia  ixx="1.0" ixy="0.0"  ixz="0.0"  iyy="0.0"  iyz="0.0"
-	izz="0.0" />
+	<inertia  ixx="1.0" ixy="0.0"  ixz="0.0"  iyy="0.0"  iyz="0.0" izz="0.0" />
       </inertial>
       <visual>
@@ -34,6 +33,5 @@
       <insert_block name="origin" />
       <axis xyz="0 1 0" />
-      <limit lower="-0.52359877559829882" upper="0.17453292519943295"
-      effort="10" velocity="1.0"/>
+      <limit lower="-0.52359877559829882" upper="0.17453292519943295" effort="10" velocity="1.0"/>
       <dynamics damping="50.5"/>
     </joint>

File: model/robots/xacro/arm_and_hand_motor.urdf.xacro (robot description, xacro)
@@ -18,12 +18,8 @@
   <xacro:sr_arm_motor>
   </xacro:sr_arm_motor>
-  <joint name="arm_link" type="revolute">
+  <joint name="arm_link" type="fixed">
     <parent link="shadowarm_handsupport_motor"/>
     <child link="forearm_motor"/>
-    <origin xyz="0 0 0" rpy="0 0 ${2.36}" />
-    <axis xyz="0 -1 0" />
-    <limit lower="0" upper="0" effort="10"
-    velocity="1.0" />
-    <dynamics damping="3.5"/>
+    <origin xyz="0 0 0" rpy="0 0 ${2.35619449}" />
   </joint>
   <xacro:shadowhand_motor>

Commit message: Remove seperate file for left hand and replace with macro so we now have:  * xacro:shadowhand_motor  * xacro:shadowhand_left_motor With the only file seperation at the top level for use in launch file to fill param:  * model/robots/xacro/shadowhand_motor.urdf.xacro  * model/robots/xacro/shadowhand_left_motor.urdf.xacro

File: model/hand_urdf/full_hand_motor.urdf.xacro (robot description, xacro)
@@ -9,4 +9,5 @@
   <include filename="$(find sr_hand)/model/hand_urdf/finger/little_finger.urdf.xacro" />
   <include filename="$(find sr_hand)/model/hand_urdf/thumb/thumb.urdf.xacro" />
+  <!-- Right Hand -->
   <xacro:macro name="shadowhand_motor">
     <xacro:forearm_motor>
@@ -34,3 +35,29 @@
     </xacro:thumb>
   </xacro:macro>
+  <!-- Left Hand -->
+  <xacro:macro name="shadowhand_left_motor">
+    <xacro:forearm_motor>
+    </xacro:forearm_motor>
+    <xacro:wrist_left parent="forearm_motor">
+      <origin xyz="0 -0.010 0.213" rpy="0 0 0" />
+    </xacro:wrist_left>
+    <xacro:palm_left parent="wrist">
+    </xacro:palm_left>
+    <xacro:finger link_prefix="ff" joint_prefix="FF" parent="palm">
+      <origin xyz="-0.033 0 0.095" rpy="0 0 0" />
+      <axis xyz="0 -1 0" />
+    </xacro:finger>
+    <xacro:finger link_prefix="mf" joint_prefix="MF" parent="palm">
+      <origin xyz="-0.011 0 0.099" rpy="0 0 0" />
+      <axis xyz="0 -1 0" />
+    </xacro:finger>
+    <xacro:finger link_prefix="rf" joint_prefix="RF" parent="palm">
+      <origin xyz="0.011 0 0.095" rpy="0 0 0" />
+      <axis xyz="0 1 0" />
+    </xacro:finger>
+    <xacro:little_finger_left link_prefix="lf" joint_prefix="LF" parent="palm">
+    </xacro:little_finger_left>
+    <xacro:thumb_left parent="palm">
+    </xacro:thumb_left>
+  </xacro:macro>
 </robot>

File: model/robots/xacro/shadowhand_left_motor.urdf.xacro (robot description, xacro)
@@ -5,7 +5,7 @@
        name="shadowhand_motor">
   <include filename="$(find sr_hand)/model/materials.urdf.xacro" />
-  <include filename="$(find sr_hand)/model/hand_urdf/full_hand_left_motor.urdf.xacro" />
+  <include filename="$(find sr_hand)/model/hand_urdf/full_hand_motor.urdf.xacro" />
   <include filename="$(find sr_hand)/model/gazebo/gazebo.urdf.xacro" />
-  <xacro:shadowhand_motor>
-  </xacro:shadowhand_motor>
+  <xacro:shadowhand_left_motor>
+  </xacro:shadowhand_left_motor>
 </robot>
