Commit message: Left handed muscle hand.
Quick test that the macros expand properly letting you stick a left hand on the
muscle base. They do :)

File: model/hand_urdf/full_hand_muscle.urdf.xacro (robot description, xacro)
@@ -9,4 +9,5 @@
   <include filename="$(find sr_hand)/model/hand_urdf/finger/little_finger.urdf.xacro" />
   <include filename="$(find sr_hand)/model/hand_urdf/thumb/thumb.urdf.xacro" />
+  <!-- Right Hand -->
   <xacro:macro name="shadowhand_muscle">
     <xacro:forearm_muscle>
@@ -34,3 +35,29 @@
     </xacro:thumb>
   </xacro:macro>
+  <!-- Left Hand -->
+  <xacro:macro name="shadowhand_left_muscle">
+    <xacro:forearm_muscle>
+    </xacro:forearm_muscle>
+    <xacro:wrist_left parent="forearm_muscle">
+      <origin xyz="0 0 0.396" rpy="0 0 0" />
+    </xacro:wrist_left>
+    <xacro:palm_left parent="wrist">
+    </xacro:palm_left>
+    <xacro:finger link_prefix="ff" joint_prefix="FF" parent="palm">
+      <origin xyz="-0.033 0 0.095" rpy="0 0 0" />
+      <axis xyz="0 -1 0" />
+    </xacro:finger>
+    <xacro:finger link_prefix="mf" joint_prefix="MF" parent="palm">
+      <origin xyz="-0.011 0 0.099" rpy="0 0 0" />
+      <axis xyz="0 -1 0" />
+    </xacro:finger>
+    <xacro:finger link_prefix="rf" joint_prefix="RF" parent="palm">
+      <origin xyz="0.011 0 0.095" rpy="0 0 0" />
+      <axis xyz="0 1 0" />
+    </xacro:finger>
+    <xacro:little_finger_left link_prefix="lf" joint_prefix="LF" parent="palm">
+    </xacro:little_finger_left>
+    <xacro:thumb_left parent="palm">
+    </xacro:thumb_left>
+  </xacro:macro>
 </robot>
