Commit message: Added manipulation stack support for the Shadow Hand and arm. Need to test.

File: model/hand_urdf/thumb/thdistal.urdf.xacro (robot description, xacro)
@@ -49,6 +49,6 @@
       <parent link="${parent}"/>
       <child link="thdistal"/>
-      <origin xyz="0 0 0.032" rpy="0 0 0" />
-      <axis xyz="0 -1 0" />
+      <origin xyz="0 0 0.032" rpy="0 0 -1.570796327" />
+      <axis xyz="1 0 0" />
       <limit lower="0" upper="1.571" effort="10"
       velocity="1.0" />

File: model/robots/xacro/arm_and_hand_motor.urdf.xacro (robot description, xacro)
@@ -21,5 +21,5 @@
     <parent link="shadowarm_handsupport_motor"/>
     <child link="forearm_motor"/>
-    <origin xyz="0 0 0" rpy="0 0 ${M_PI}" />
+    <origin xyz="0 0 0" rpy="0 0 ${2.36}" />
     <axis xyz="0 -1 0" />
     <limit lower="0" upper="0" effort="10"

File: model/robots/xacro/desk_arm_and_hand_motor.urdf.xacro (robot description, xacro)
@@ -1,27 +1,19 @@
 <robot xmlns:xacro="http://ros.org/wiki/xacro" name="arm_and_hand">
   <include filename="$(find sr_hand)/model/materials.urdf.xacro" />
-  <include filename="$(find sr_hand)/model/arm_urdf/full_arm_muscle.urdf.xacro" />
-  <include filename="$(find sr_hand)/model/hand_urdf/full_hand_muscle.urdf.xacro" />
+  <include filename="$(find sr_hand)/model/arm_urdf/full_arm_motor.urdf.xacro" />
+  <include filename="$(find sr_hand)/model/hand_urdf/full_hand_motor.urdf.xacro" />
   <include filename="$(find sr_hand)/model/gazebo/gazebo.urdf.xacro" />
-<<<<<<< TREE
   <include filename="$(find sr_hand)/model/desk/desk.urdf.xacro" />
   <xacro:desk/>
-  <joint name="arm_to_desk_fixed" type="fixed">
+  <joint name="base_fix" type="fixed">
     <parent link="desk_pillar"/>
     <child link="shadowarm_base"/>
     <origin rpy="0 0 0" xyz="0 0 1.0"/>
   </joint>
-  <joint name="base_fix" type="fixed">
-    <parent link="world"/>
-    <child link="desk_support"/>
-    <origin rpy="0 0 0" xyz="0 0 0"/>
-  </joint>
-=======
->>>>>>> MERGE-SOURCE
-  <xacro:sr_arm_muscle>
-  </xacro:sr_arm_muscle>
+  <xacro:sr_arm_motor>
+  </xacro:sr_arm_motor>
   <joint name="arm_link" type="revolute">
-    <parent link="shadowarm_handsupport_muscle"/>
-    <child link="forearm_muscle"/>
+    <parent link="shadowarm_handsupport_motor"/>
+    <child link="forearm_motor"/>
     <origin xyz="0 0 0" rpy="0 0 ${M_PI}" />
     <axis xyz="0 -1 0" />
@@ -30,5 +22,5 @@
     <dynamics damping="3.5"/>
   </joint>
-  <xacro:shadowhand_muscle>
-  </xacro:shadowhand_muscle>
+  <xacro:shadowhand_motor>
+  </xacro:shadowhand_motor>
 </robot>
