Commit message: Refactor thbase.urdf.xacro to avoid duplication.

File: model/hand_urdf/thumb/thbase.urdf.xacro (robot description, xacro)
@@ -9,8 +9,17 @@
   <!-- Right Hand -->
   <xacro:macro name="thbase" params="parent">
+      <xacro:thbase_base parent="${parent}" reflect="1" joint_yaw="0" />
+  </xacro:macro>
+  <!-- Left Hand -->
+  <xacro:macro name="thbase_left" params="parent">
+      <xacro:thbase_base parent="${parent}" reflect="-1" joint_yaw="${M_PI}" />
+  </xacro:macro>
+  <!-- Macro to used to generate left and right handed versions.
+  DO NOT use out side of here ie treat as a private macro -->
+  <xacro:macro name="thbase_base" params="parent reflect joint_yaw">
     <link name="thbase">
       <inertial>
 	<mass value="0.010" />
-	<origin xyz="0.034 0.0085 0.029" rpy="0 0 0"/>
+    <origin xyz="${reflect*0.034} 0.0085 0.029" rpy="0 0 0"/>
 	<inertia  ixx="0.0" ixy="0.0"  ixz="0.0"  iyy="0.0"  iyz="0.0"
 	izz="0.1" />
@@ -49,56 +58,6 @@
       <parent link="${parent}"/>
       <child link="thbase"/>
-      <origin xyz="0.034 -0.0085 0.029" rpy="0 ${M_PI/4} 0" />
-      <axis xyz="0 0 -1" />
-      <limit lower="-1.047" upper="1.047" effort="10"
-      velocity="1.0" />
-      <dynamics damping="50.5"/>
-    </joint>
-    <xacro:thbase_transmission />
-  </xacro:macro>
-  <!-- Left Hand -->
-  <xacro:macro name="thbase_left" params="parent">
-    <link name="thbase">
-      <inertial>
-	<mass value="0.010" />
-	<origin xyz="-0.034 0.0085 0.029" rpy="0 0 0"/>
-	<inertia  ixx="0.0" ixy="0.0"  ixz="0.0"  iyy="0.0"  iyz="0.0"
-	izz="0.1" />
-      </inertial>
-      <visual>
-	<origin xyz="0 0 0" rpy="0 0 0" />
-	<geometry name="thbase_visual">
-	  <box size="0.001 0.001 0.001" />
-	</geometry>
-      <material name="shadow_thbase_material">
-	  <color rgba="0.5 0.5 0.5 1.0"/>
-	</material>
-      </visual>
-      <collision>
-	<origin xyz="0 0 0" rpy="0 0 0 " />
-	<geometry name="thbase_collision_geom">
-	  <box size="0.001 0.001 0.001" />
-	</geometry>
-      </collision>
-    </link>
-    <gazebo reference="thbase">
-      <sensor:contact name="thbase_contact_sensor">
-        <geom>thbase_geom</geom>
-       <updateRate>100.0</updateRate>
-        <controller:gazebo_ros_bumper name="thbase_gazebo_ros_bumper_controller" plugin="libgazebo_ros_bumper.so">
-          <alwaysOn>true</alwaysOn>
-          <updateRate>100.0</updateRate>
-          <frameName>thbase</frameName>
-          <bumperTopicName>thbase_bumper</bumperTopicName>
-          <interface:bumper name="thbase_gazebo_ros_bumper_iface" />
-        </controller:gazebo_ros_bumper>
-      </sensor:contact>
-      <material>Gazebo/Grey</material>
-    </gazebo>
-    <joint name="THJ5" type="revolute">
-      <parent link="${parent}"/>
-      <child link="thbase"/>
-      <origin xyz="-0.034 -0.0085 0.029" rpy="0 ${M_PI/4} ${M_PI}" />
-      <axis xyz="0 0 1" />
+      <origin xyz="${reflect*0.034} -0.0085 0.029" rpy="0 ${M_PI/4} ${joint_yaw}" />
+      <axis xyz="0 0 ${reflect*-1}" />
       <limit lower="-1.047" upper="1.047" effort="10"
       velocity="1.0" />
