Commit message: Added a hand_controller dedicated to gazebo simulation (because controllers settings may not be the same) Corrected gazebo_arm_and_hand_motor.launch to use it Corrected forearm_motor inertia to a more correct one (cyl of 4kg height 444mm, radius 60mm)

File: model/hand_urdf/forearm/forearm_motor.urdf.xacro (robot description, xacro)
@@ -4,7 +4,7 @@
     <link name="forearm_motor">
       <inertial>
-	<origin xyz="0 0 0" />
-	<mass value="3.0" />
-	<inertia  ixx="1.0" ixy="0.0"  ixz="0.0"  iyy="0.0"  iyz="0.0"  izz="0.0" />
+	<origin xyz="0 0 0.12" />
+	<mass value="4.0" />
+	<inertia  ixx="0.06813" ixy="0.0"  ixz="0.0"  iyy="0.06813"  iyz="0.0"  izz="0.0072" />
       </inertial>
       <visual>

Commit message: Re-added the full robot publisher (required for markers and other stacks) Corrected sr_arm_motor_finger_ik.launch transform of shadowarm_base to be the same as sr_arm_motor.launch Changed forearm weight (fake weight was really to heavy), and adapted arm_controller gains to move the arm quite correctly Corrected a bug in shadowhand_ros.py to handle missing hand when calling valueof Added sr_bumper_rviz_markers to tactile (to see bumper forces in rviz) Corrected sr_gazebo_virtual_tactile_sensor to now use a sum of all contact force instead of only one contact force, also publish zero if no data received (should be already corrected in recent ROS bumpers) Corrected ordered joint merger (pos and target) that were not doing their job

File: model/hand_urdf/forearm/forearm_motor.urdf.xacro (robot description, xacro)
@@ -5,5 +5,5 @@
       <inertial>
 	<origin xyz="0 0 0" />
-	<mass value="30.0" />
+	<mass value="15.0" />
 	<inertia  ixx="10.8" ixy="0.0"  ixz="0.0"  iyy="10.8"  iyz="0.0"  izz="5.4" />
       </inertial>
