Commit message: Reworked on inertia of the arm and hand to get more stability (but less correlation to real world values...). Forearm has its original weight back as inertia seem to solve our problems, not mass.

File: model/arm_urdf/trunk/shadowarm_trunk.urdf.xacro (robot description, xacro)
@@ -5,6 +5,6 @@
 	<inertial>
 	  <origin xyz="0 0 0.27025" rpy="0 0 0" />
-	  <mass value="5" />
-	  <inertia  ixx="1.0" ixy="0.0"  ixz="0.0"  iyy="0.0"  iyz="0.0"  izz="0.0" />
+	  <mass value="10" />
+	  <inertia  ixx="1.47" ixy="0.0"  ixz="0.0"  iyy="1.47"  iyz="0.0"  izz="2.4" />
 	</inertial>
 	<visual>

File: model/arm_urdf/upper_arm/shadowarm_upperarm.urdf.xacro (robot description, xacro)
@@ -6,5 +6,5 @@
 	<origin xyz="0 -0.067 -0.1845" rpy="0 0 0" />
 	<mass value="2" />
-	<inertia  ixx="1.0" ixy="0.0"  ixz="0.0"  iyy="0.0"  iyz="0.0"  izz="0.0" />
+	<inertia  ixx="0.5" ixy="0.0"  ixz="0.0"  iyy="0.5"  iyz="0.0"  izz="0.1" />
       </inertial>
       <visual>

File: model/hand_urdf/finger/distal/distal.urdf.xacro (robot description, xacro)
@@ -12,5 +12,5 @@
 	<mass value="0.010" />
 	<origin xyz="0 0 0.025" />
-	<inertia  ixx="1.0" ixy="0.0"  ixz="0.0"  iyy="0.0"  iyz="0.0"
+	<inertia  ixx="0.1" ixy="0.0"  ixz="0.0"  iyy="0.1"  iyz="0.0"
 	izz="0.0" />
       </inertial>

File: model/hand_urdf/finger/knuckle/knuckle.urdf.xacro (robot description, xacro)
@@ -13,5 +13,5 @@
 	<insert_block name="origin" />
 	<mass value="0.008" />
-	<inertia  ixx="1.0" ixy="0.0"  ixz="0.0"  iyy="0.0"  iyz="0.0"
+	<inertia  ixx="0.0" ixy="0.0"  ixz="0.0"  iyy="0.1"  iyz="0.0"
 	izz="0.0" />
       </inertial>

File: model/hand_urdf/finger/lfmetacarpal/lfmetacarpal.urdf.xacro (robot description, xacro)
@@ -12,6 +12,6 @@
 	<origin xyz="-0.033 0 0.02071" rpy="0 0 0" />
 	<mass value="0.075" />
-	<inertia  ixx="1.0" ixy="0.0"  ixz="0.0"  iyy="0.0"  iyz="0.0"
-	izz="0.0" />
+	<inertia  ixx="0.1" ixy="0.0"  ixz="0.0"  iyy="0.1"  iyz="0.0"
+	izz="0.1" />
       </inertial>
       <visual>

File: model/hand_urdf/finger/little_finger.urdf.xacro (robot description, xacro)
@@ -18,6 +18,6 @@
 	<origin xyz="0 0 0.06579" rpy="0 0 0" />
 	<mass value="0.008" />
-	<inertia  ixx="1.0" ixy="0.0"  ixz="0.0"  iyy="0.0"  iyz="0.0"
-	izz="0.0" />
+	<inertia  ixx="0.1" ixy="0.0"  ixz="0.0"  iyy="0.1"  iyz="0.0"
+	izz="0.1" />
       </inertial>
       <visual>

File: model/hand_urdf/finger/middle/middle.urdf.xacro (robot description, xacro)
@@ -12,5 +12,5 @@
 	<origin xyz="0 0 0.045" rpy="0 0 0" />
 	<mass value="0.012" />
-	<inertia  ixx="1.0" ixy="0.0"  ixz="0.0"  iyy="0.0"  iyz="0.0"
+	<inertia  ixx="0.1" ixy="0.0"  ixz="0.0"  iyy="0.1"  iyz="0.0"
 	izz="0.0" />
       </inertial>

File: model/hand_urdf/finger/proximal/proximal.urdf.xacro (robot description, xacro)
@@ -12,5 +12,5 @@
 	<mass value="0.014" />
 	<origin xyz="0 0 0" />
-	<inertia  ixx="1.0" ixy="0.0"  ixz="0.0"  iyy="0.0"  iyz="0.0"
+	<inertia  ixx="0.1" ixy="0.0"  ixz="0.0"  iyy="0.1"  iyz="0.0"
 	izz="0.0" />
       </inertial>

File: model/hand_urdf/forearm/forearm_motor.urdf.xacro (robot description, xacro)
@@ -5,6 +5,6 @@
       <inertial>
 	<origin xyz="0 0 0" />
-	<mass value="15.0" />
-	<inertia  ixx="10.8" ixy="0.0"  ixz="0.0"  iyy="10.8"  iyz="0.0"  izz="5.4" />
+	<mass value="3.0" />
+	<inertia  ixx="1.0" ixy="0.0"  ixz="0.0"  iyy="1.0"  iyz="0.0"  izz="1.0" />
       </inertial>
       <visual>

File: model/hand_urdf/palm/palm.urdf.xacro (robot description, xacro)
@@ -12,5 +12,5 @@
 	<origin xyz="0 0 0.247" rpy="0 0 0" />
 	<mass value="0.3" />
-	<inertia  ixx="1.266" ixy="0.0"  ixz="0.0"  iyy="1.436"  iyz="0.0"	izz="0.19" />
+	<inertia  ixx="0.5" ixy="0.0"  ixz="0.0"  iyy="0.5"  iyz="0.0"	izz="0.3" />
       </inertial>
       <visual>
@@ -49,5 +49,5 @@
       <limit lower="-0.78539816339744828" upper="0.6108652381980153"
       effort="1" velocity="0.2"/>
-      <dynamics damping="50.5"/>
+      <dynamics damping="200.5"/>
     </joint>
     <xacro:shadowhand_palm_transmission />

File: model/hand_urdf/thumb/thbase.urdf.xacro (robot description, xacro)
@@ -12,6 +12,6 @@
 	<mass value="0.010" />
 	<origin xyz="0.034 0.0085 0.029" rpy="0 0 0"/>
-	<inertia  ixx="1.0" ixy="0.0"  ixz="0.0"  iyy="0.0"  iyz="0.0"
-	izz="0.0" />
+	<inertia  ixx="0.0" ixy="0.0"  ixz="0.0"  iyy="0.0"  iyz="0.0"
+	izz="0.1" />
       </inertial>
       <visual>

File: model/hand_urdf/thumb/thdistal.urdf.xacro (robot description, xacro)
@@ -12,6 +12,6 @@
 	<mass value="0.016" />
 	<origin xyz="-0.02263 0 0.02263" rpy="0 0 0"/>
-	<inertia  ixx="1.0" ixy="0.0"  ixz="0.0"  iyy="0.0"  iyz="0.0"
-	izz="0.0" />
+	<inertia  ixx="0.1" ixy="0.0"  ixz="0.0"  iyy="0.1"  iyz="0.0"
+	izz="0.1" />
       </inertial>
       <visual>

File: model/hand_urdf/thumb/thhub.urdf.xacro (robot description, xacro)
@@ -12,6 +12,6 @@
 	<mass value="0.002" />
 	<origin xyz="0.02687 0 0.02687" rpy="0 0 0"/>
-	<inertia  ixx="1.0" ixy="0.0"  ixz="0.0"  iyy="0.0"  iyz="0.0"
-	izz="0.0" />
+	<inertia  ixx="0.1" ixy="0.0"  ixz="0.0"  iyy="0.1"  iyz="0.0"
+	izz="0.1" />
       </inertial>
       <visual>

File: model/hand_urdf/thumb/thmiddle.urdf.xacro (robot description, xacro)
@@ -12,6 +12,6 @@
 	<mass value="0.016" />
 	<origin xyz="0 0 0" rpy="0 0 0"/>
-	<inertia  ixx="1.0" ixy="0.0"  ixz="0.0"  iyy="0.0"  iyz="0.0"
-	izz="0.0" />
+	<inertia  ixx="0.1" ixy="0.0"  ixz="0.0"  iyy="0.1"  iyz="0.0"
+	izz="0.1" />
       </inertial>
       <visual>

File: model/hand_urdf/thumb/thproximal.urdf.xacro (robot description, xacro)
@@ -12,6 +12,5 @@
 	<mass value="0.016" />
 	<origin xyz="0 0 0" rpy="0 0 0"/>
-	<inertia  ixx="1.0" ixy="0.0"  ixz="0.0"  iyy="0.0"  iyz="0.0"
-	izz="0.0" />
+	<inertia  ixx="0.1" ixy="0.0"  ixz="0.0"  iyy="0.1"  iyz="0.0"	izz="0.1" />
       </inertial>
       <visual>

File: model/hand_urdf/wrist/wrist.urdf.xacro (robot description, xacro)
@@ -34,5 +34,5 @@
       <axis xyz="0 1 0" />
       <limit lower="-0.52359877559829882" upper="0.17453292519943295" effort="1" velocity="0.2"/>
-      <dynamics damping="50.5"/>
+      <dynamics damping="200.5"/>
     </joint>
     <xacro:shadowhand_wrist_transmission />
