Commit message: Renamed arm_controllers Created a CAN_compatibility_arm node to route the sendupdate messages for to arm to arm_controllers Changed some settings in urdf cause wrist is was too slow

File: model/hand_urdf/palm/palm.urdf.xacro (robot description, xacro)
@@ -48,6 +48,6 @@
       <axis xyz="1 0 0" />
       <limit lower="-0.78539816339744828" upper="0.6108652381980153"
-      effort="1" velocity="0.2"/>
-      <dynamics damping="200.5"/>
+      effort="5" velocity="1.0"/>
+      <dynamics damping="100.5"/>
     </joint>
     <xacro:shadowhand_palm_transmission />

File: model/hand_urdf/wrist/wrist.urdf.xacro (robot description, xacro)
@@ -33,6 +33,6 @@
       <insert_block name="origin" />
       <axis xyz="0 1 0" />
-      <limit lower="-0.52359877559829882" upper="0.17453292519943295" effort="1" velocity="0.2"/>
-      <dynamics damping="200.5"/>
+      <limit lower="-0.52359877559829882" upper="0.17453292519943295" effort="5" velocity="1.0"/>
+      <dynamics damping="100.5"/>
     </joint>
     <xacro:shadowhand_wrist_transmission />
