Commit message: Tidy up XML so indents makes sense.

File: model/hand_urdf/finger/little_finger.urdf.xacro (robot description, xacro)
@@ -12,25 +12,24 @@
   <include filename="$(find sr_hand)/model/hand_urdf/finger/lfmetacarpal/lfmetacarpal.urdf.xacro" />
   <xacro:macro name="little_finger" params="link_prefix joint_prefix parent">
-    <xacro:lfmetacarpal parent="${parent}" >
+    <xacro:lfmetacarpal parent="${parent}">
     </xacro:lfmetacarpal>
     <link name="lfknuckle">
       <inertial>
-	<origin xyz="0 0 0.06579" rpy="0 0 0" />
-	<mass value="0.008" />
-	<inertia  ixx="0.1" ixy="0.0"  ixz="0.0"  iyy="0.1"  iyz="0.0"
-	izz="0.1" />
+        <origin xyz="0 0 0.06579" rpy="0 0 0" />
+        <mass value="0.008" />
+        <inertia ixx="0.1" ixy="0.0" ixz="0.0" iyy="0.1" iyz="0.0" izz="0.1" />
       </inertial>
       <visual>
-	<origin xyz="0 0 0" rpy="0 0 0" />
-	<geometry name="knuckle_visual">
-      <mesh filename="package://sr_hand/model/meshes/knuckle.mesh" scale="0.001 0.001 0.001" />
-      </geometry>
-      <material name="LightGrey" />
+        <origin xyz="0 0 0" rpy="0 0 0" />
+        <geometry name="knuckle_visual">
+          <mesh filename="package://sr_hand/model/meshes/knuckle.mesh" scale="0.001 0.001 0.001" />
+        </geometry>
+        <material name="LightGrey" />
       </visual>
       <collision>
-	<origin xyz="0 0 0" rpy="0 0 0" />
-	<geometry name="knuckle_collision_geom">
-	  <box size="0.005 0.005 0.005" />
-	</geometry>
+        <origin xyz="0 0 0" rpy="0 0 0" />
+        <geometry name="knuckle_collision_geom">
+          <box size="0.005 0.005 0.005" />
+        </geometry>
       </collision>
     </link>
@@ -38,5 +37,5 @@
       <sensor:contact name="lfknuckle_contact_sensor">
         <geom>lfknuckle_geom</geom>
-       <updateRate>100.0</updateRate>
+        <updateRate>100.0</updateRate>
         <controller:gazebo_ros_bumper name="lfknuckle_gazebo_ros_bumper_controller" plugin="libgazebo_ros_bumper.so">
           <alwaysOn>true</alwaysOn>
@@ -50,11 +49,10 @@
     </gazebo>
     <joint name="LFJ4" type="revolute">
-      <parent link="lfmetacarpal"/>
-      <child link="lfknuckle"/>
+      <parent link="lfmetacarpal" />
+      <child link="lfknuckle" />
       <origin xyz="0 0 0.06579" rpy="0 0 0" />
       <axis xyz="0 1 0" />
-      <limit lower="-0.43633231299858238" upper="0.43633231299858238"
-      effort="10" velocity="1.0"/>
-      <dynamics damping="50.5"/>
+      <limit lower="-0.43633231299858238" upper="0.43633231299858238" effort="10" velocity="1.0" />
+      <dynamics damping="50.5" />
     </joint>
     <transmission type="sr_mechanism_model/SimpleTransmission" name="lfknuckle_transmission">
@@ -65,9 +63,9 @@
       <pulsesPerRevolution>90000</pulsesPerRevolution>
     </transmission>
-    <xacro:proximal link_prefix="${link_prefix}" joint_prefix="${joint_prefix}" parent="${link_prefix}knuckle" >
+    <xacro:proximal link_prefix="${link_prefix}" joint_prefix="${joint_prefix}" parent="${link_prefix}knuckle">
     </xacro:proximal>
-    <xacro:middle link_prefix="${link_prefix}" joint_prefix="${joint_prefix}" parent="${link_prefix}proximal" >
+    <xacro:middle link_prefix="${link_prefix}" joint_prefix="${joint_prefix}" parent="${link_prefix}proximal">
     </xacro:middle>
-    <xacro:distal link_prefix="${link_prefix}" joint_prefix="${joint_prefix}" parent="${link_prefix}middle" >
+    <xacro:distal link_prefix="${link_prefix}" joint_prefix="${joint_prefix}" parent="${link_prefix}middle">
     </xacro:distal>
   </xacro:macro>
