Commit message: Added more precision to LFJ5 axis in urdf

File: model/hand_urdf/finger/lfmetacarpal/lfmetacarpal.urdf.xacro (robot description, xacro)
@@ -47,5 +47,5 @@
       <child link="lfmetacarpal"/>
       <origin xyz="-0.033 0 0.02071" rpy="0 0 0" />
-      <axis xyz="0.57 0 0.82" />
+      <axis xyz="0.573576436 0 0.819152044" />
       <limit lower="0" upper="0.69813170079773179" effort="10"
       velocity="1.0" />

Commit message: Start to paramatise the origin for the little finger.

File: model/hand_urdf/finger/lfmetacarpal/lfmetacarpal.urdf.xacro (robot description, xacro)
@@ -7,11 +7,10 @@
        xmlns:geom="http://playerstage.sourceforge.net/gazebo/xmlschema/#geom">
   <include filename="$(find sr_hand)/model/hand_urdf/finger/lfmetacarpal/lfmetacarpal.transmission.xacro" />
-  <xacro:macro name="lfmetacarpal" params="parent">
+  <xacro:macro name="lfmetacarpal" params="parent *origin">
     <link name="lfmetacarpal">
       <inertial>
-	<origin xyz="-0.033 0 0.02071" rpy="0 0 0" />
-	<mass value="0.075" />
-	<inertia  ixx="0.1" ixy="0.0"  ixz="0.0"  iyy="0.1"  iyz="0.0"
-	izz="0.1" />
+        <insert_block name="origin" />
+        <mass value="0.075" />
+        <inertia  ixx="0.1" ixy="0.0"  ixz="0.0"  iyy="0.1"  iyz="0.0" izz="0.1" />
       </inertial>
       <visual>

File: model/hand_urdf/finger/little_finger.urdf.xacro (robot description, xacro)
@@ -13,4 +13,5 @@
   <xacro:macro name="little_finger" params="link_prefix joint_prefix parent">
     <xacro:lfmetacarpal parent="${parent}">
+      <origin xyz="-0.033 0 0.02071" rpy="0 0 0" />
     </xacro:lfmetacarpal>
     <link name="lfknuckle">

Commit message: Paramatise the little finger origin.
May not be the right approach, as may need to fix up the axis of the the LFJ5
joing as well. Which with this setup will need the axis block passing in as
well. However all we do is flip the x cord on the origin and axis so a reflect
param (1|-1) might be better as we will never need more than one little finger.
Can test that after creating a mirrored mesh for the joint.

File: model/hand_urdf/finger/lfmetacarpal/lfmetacarpal.urdf.xacro (robot description, xacro)
@@ -45,5 +45,5 @@
       <parent link="${parent}"/>
       <child link="lfmetacarpal"/>
-      <origin xyz="-0.033 0 0.02071" rpy="0 0 0" />
+      <insert_block name="origin" />
       <axis xyz="0.573576436 0 0.819152044" />
       <limit lower="0" upper="0.69813170079773179" effort="10"

File: model/hand_urdf/finger/little_finger.urdf.xacro (robot description, xacro)
@@ -11,7 +11,7 @@
   <include filename="$(find sr_hand)/model/hand_urdf/finger/distal/distal.urdf.xacro" />
   <include filename="$(find sr_hand)/model/hand_urdf/finger/lfmetacarpal/lfmetacarpal.urdf.xacro" />
-  <xacro:macro name="little_finger" params="link_prefix joint_prefix parent">
+  <xacro:macro name="little_finger" params="link_prefix joint_prefix parent *origin">
     <xacro:lfmetacarpal parent="${parent}">
-      <origin xyz="-0.033 0 0.02071" rpy="0 0 0" />
+      <insert_block name="origin" />
     </xacro:lfmetacarpal>
     <link name="lfknuckle">

File: model/hand_urdf/full_hand_motor.urdf.xacro (robot description, xacro)
@@ -30,4 +30,5 @@
     </xacro:finger>
     <xacro:little_finger link_prefix="lf" joint_prefix="LF" parent="palm">
+      <origin xyz="-0.033 0 0.02071" rpy="0 0 0" />
     </xacro:little_finger>
     <xacro:thumb parent="palm">

File: model/hand_urdf/full_hand_muscle.urdf.xacro (robot description, xacro)
@@ -30,4 +30,5 @@
     </xacro:finger>
     <xacro:little_finger link_prefix="lf" joint_prefix="LF" parent="palm">
+      <origin xyz="-0.033 0 0.02071" rpy="0 0 0" />
     </xacro:little_finger>
     <xacro:thumb parent="palm">

Commit message: Finish left little finger.
Back out changes 327..326 (paramatised little finger origin) and try different
approach, named macro little_finger_left (that uses lfmetacarpal_left). Works
well. Also adds mirrored mesh for lfmetacarpal. Joint LFJ5 moves correctly.

File: model/hand_urdf/finger/lfmetacarpal/lfmetacarpal.urdf.xacro (robot description, xacro)
@@ -7,10 +7,12 @@
        xmlns:geom="http://playerstage.sourceforge.net/gazebo/xmlschema/#geom">
   <include filename="$(find sr_hand)/model/hand_urdf/finger/lfmetacarpal/lfmetacarpal.transmission.xacro" />
-  <xacro:macro name="lfmetacarpal" params="parent *origin">
+  <!-- Right Handed -->
+  <xacro:macro name="lfmetacarpal" params="parent">
     <link name="lfmetacarpal">
       <inertial>
-        <insert_block name="origin" />
-        <mass value="0.075" />
-        <inertia  ixx="0.1" ixy="0.0"  ixz="0.0"  iyy="0.1"  iyz="0.0" izz="0.1" />
+	<origin xyz="-0.033 0 0.02071" rpy="0 0 0" />
+	<mass value="0.075" />
+	<inertia  ixx="0.1" ixy="0.0"  ixz="0.0"  iyy="0.1"  iyz="0.0"
+	izz="0.1" />
       </inertial>
       <visual>
@@ -45,5 +47,5 @@
       <parent link="${parent}"/>
       <child link="lfmetacarpal"/>
-      <insert_block name="origin" />
+      <origin xyz="-0.033 0 0.02071" rpy="0 0 0" />
       <axis xyz="0.573576436 0 0.819152044" />
       <limit lower="0" upper="0.69813170079773179" effort="10"
@@ -53,3 +55,51 @@
     <xacro:lfmetacarpal_transmission />
   </xacro:macro>
+  <!-- Left Handed -->
+  <xacro:macro name="lfmetacarpal_left" params="parent">
+    <link name="lfmetacarpal">
+      <inertial>
+	<origin xyz="0.033 0 0.02071" rpy="0 0 0" />
+	<mass value="0.075" />
+	<inertia  ixx="0.1" ixy="0.0"  ixz="0.0"  iyy="0.1"  iyz="0.0"
+	izz="0.1" />
+      </inertial>
+      <visual>
+	<origin xyz="0 0 0" rpy="0 0 0" />
+	<geometry name="lfmetacarpal_visual">
+	  <mesh filename="package://sr_hand/model/meshes/lfmetacarpal_left.mesh" scale="0.001 0.001 0.001" />
+	</geometry>
+	<material name="Grey" />
+      </visual>
+      <collision>
+	<origin xyz="0.015 0 0.015" rpy="0 0 0" />
+	<geometry name="lfmetacarpal_collision_geom">
+	  <box size="0.005 0.005 0.03" />
+	</geometry>
+      </collision>
+    </link>
+    <gazebo reference="lfmetacarpal">
+      <sensor:contact name="lfmetacarpal_contact_sensor">
+        <geom>lfmetacarpal_geom</geom>
+       <updateRate>100.0</updateRate>
+        <controller:gazebo_ros_bumper name="lfmetacarpal_gazebo_ros_bumper_controller" plugin="libgazebo_ros_bumper.so">
+          <alwaysOn>true</alwaysOn>
+          <updateRate>100.0</updateRate>
+          <frameName>lfmetacarpal</frameName>
+          <bumperTopicName>lfmetacarpal_bumper</bumperTopicName>
+          <interface:bumper name="lfmetacarpal_gazebo_ros_bumper_iface" />
+        </controller:gazebo_ros_bumper>
+      </sensor:contact>
+      <material>Gazebo/Grey</material>
+    </gazebo>
+    <joint name="LFJ5" type="revolute">
+      <parent link="${parent}"/>
+      <child link="lfmetacarpal"/>
+      <origin xyz="0.033 0 0.02071" rpy="0 0 0" />
+      <axis xyz="0.573576436 0 -0.819152044" />
+      <limit lower="0" upper="0.69813170079773179" effort="10"
+      velocity="1.0" />
+      <dynamics damping="50.5"/>
+    </joint>
+    <xacro:lfmetacarpal_transmission />
+  </xacro:macro>
 </robot>

File: model/hand_urdf/finger/little_finger.urdf.xacro (robot description, xacro)
@@ -11,7 +11,7 @@
   <include filename="$(find sr_hand)/model/hand_urdf/finger/distal/distal.urdf.xacro" />
   <include filename="$(find sr_hand)/model/hand_urdf/finger/lfmetacarpal/lfmetacarpal.urdf.xacro" />
-  <xacro:macro name="little_finger" params="link_prefix joint_prefix parent *origin">
+  <!-- Right Handed -->
+  <xacro:macro name="little_finger" params="link_prefix joint_prefix parent">
     <xacro:lfmetacarpal parent="${parent}">
-      <insert_block name="origin" />
     </xacro:lfmetacarpal>
     <link name="lfknuckle">
@@ -71,3 +71,63 @@
     </xacro:distal>
   </xacro:macro>
+  <!-- Left Handed -->
+  <xacro:macro name="little_finger_left" params="link_prefix joint_prefix parent">
+    <xacro:lfmetacarpal_left parent="${parent}">
+    </xacro:lfmetacarpal_left>
+    <link name="lfknuckle">
+      <inertial>
+        <origin xyz="0 0 0.06579" rpy="0 0 0" />
+        <mass value="0.008" />
+        <inertia ixx="0.1" ixy="0.0" ixz="0.0" iyy="0.1" iyz="0.0" izz="0.1" />
+      </inertial>
+      <visual>
+        <origin xyz="0 0 0" rpy="0 0 0" />
+        <geometry name="knuckle_visual">
+          <mesh filename="package://sr_hand/model/meshes/knuckle.mesh" scale="0.001 0.001 0.001" />
+        </geometry>
+        <material name="LightGrey" />
+      </visual>
+      <collision>
+        <origin xyz="0 0 0" rpy="0 0 0" />
+        <geometry name="knuckle_collision_geom">
+          <box size="0.005 0.005 0.005" />
+        </geometry>
+      </collision>
+    </link>
+    <gazebo reference="lfknuckle">
+      <sensor:contact name="lfknuckle_contact_sensor">
+        <geom>lfknuckle_geom</geom>
+        <updateRate>100.0</updateRate>
+        <controller:gazebo_ros_bumper name="lfknuckle_gazebo_ros_bumper_controller" plugin="libgazebo_ros_bumper.so">
+          <alwaysOn>true</alwaysOn>
+          <updateRate>100.0</updateRate>
+          <frameName>lfknuckle</frameName>
+          <bumperTopicName>lfknuckle_bumper</bumperTopicName>
+          <interface:bumper name="lfknuckle_gazebo_ros_bumper_iface" />
+        </controller:gazebo_ros_bumper>
+      </sensor:contact>
+      <material>PR2/Grey2</material>
+    </gazebo>
+    <joint name="LFJ4" type="revolute">
+      <parent link="lfmetacarpal" />
+      <child link="lfknuckle" />
+      <origin xyz="0 0 0.06579" rpy="0 0 0" />
+      <axis xyz="0 1 0" />
+      <limit lower="-0.43633231299858238" upper="0.43633231299858238" effort="10" velocity="1.0" />
+      <dynamics damping="50.5" />
+    </joint>
+    <transmission type="sr_mechanism_model/SimpleTransmission" name="lfknuckle_transmission">
+      <actuator name="LFJ4" />
+      <joint name="LFJ4" />
+      <mechanicalReduction>1</mechanicalReduction>
+      <motorTorqueConstant>1</motorTorqueConstant>
+      <pulsesPerRevolution>90000</pulsesPerRevolution>
+    </transmission>
+    <xacro:proximal link_prefix="${link_prefix}" joint_prefix="${joint_prefix}" parent="${link_prefix}knuckle">
+    </xacro:proximal>
+    <xacro:middle link_prefix="${link_prefix}" joint_prefix="${joint_prefix}" parent="${link_prefix}proximal">
+    </xacro:middle>
+    <xacro:distal link_prefix="${link_prefix}" joint_prefix="${joint_prefix}" parent="${link_prefix}middle">
+    </xacro:distal>
+  </xacro:macro>
 </robot>

File: model/hand_urdf/full_hand_left_motor.urdf.xacro (robot description, xacro)
@@ -31,7 +31,6 @@
       <axis xyz="0 1 0" />
     </xacro:finger>
-    <xacro:little_finger link_prefix="lf" joint_prefix="LF" parent="palm">
-      <origin xyz="0.033 0 0.02071" rpy="0 0 0" />
-    </xacro:little_finger>
+    <xacro:little_finger_left link_prefix="lf" joint_prefix="LF" parent="palm">
+    </xacro:little_finger_left>
     <!--
     <xacro:thumb parent="palm">

File: model/hand_urdf/full_hand_motor.urdf.xacro (robot description, xacro)
@@ -30,5 +30,4 @@
     </xacro:finger>
     <xacro:little_finger link_prefix="lf" joint_prefix="LF" parent="palm">
-      <origin xyz="-0.033 0 0.02071" rpy="0 0 0" />
     </xacro:little_finger>
     <xacro:thumb parent="palm">

File: model/hand_urdf/full_hand_muscle.urdf.xacro (robot description, xacro)
@@ -30,5 +30,4 @@
     </xacro:finger>
     <xacro:little_finger link_prefix="lf" joint_prefix="LF" parent="palm">
-      <origin xyz="-0.033 0 0.02071" rpy="0 0 0" />
     </xacro:little_finger>
     <xacro:thumb parent="palm">

Commit message: Refactor - remove the left/right hand duplication in little finger files using macros.

File: model/hand_urdf/finger/lfmetacarpal/lfmetacarpal.urdf.xacro (robot description, xacro)
@@ -9,23 +9,31 @@
   <!-- Right Handed -->
   <xacro:macro name="lfmetacarpal" params="parent">
+      <xacro:lfmetacarpal_base parent="${parent}" reflect="1" mesh="lfmetacarpal.mesh" />
+  </xacro:macro>
+  <!-- Left Handed -->
+  <xacro:macro name="lfmetacarpal_left" params="parent">
+      <xacro:lfmetacarpal_base parent="${parent}" reflect="-1" mesh="lfmetacarpal_left.mesh" />
+  </xacro:macro>
+  <!-- Macro to used to generate left and right handed versions.
+  DO NOT use out side of here ie treat as a private macro -->
+  <xacro:macro name="lfmetacarpal_base" params="parent reflect mesh">
     <link name="lfmetacarpal">
       <inertial>
-	<origin xyz="-0.033 0 0.02071" rpy="0 0 0" />
-	<mass value="0.075" />
-	<inertia  ixx="0.1" ixy="0.0"  ixz="0.0"  iyy="0.1"  iyz="0.0"
-	izz="0.1" />
+        <origin xyz="${reflect*-0.033} 0 0.02071" rpy="0 0 0" />
+	    <mass value="0.075" />
+	    <inertia  ixx="0.1" ixy="0.0"  ixz="0.0"  iyy="0.1"  iyz="0.0" izz="0.1" />
       </inertial>
       <visual>
-	<origin xyz="0 0 0" rpy="0 0 0" />
-	<geometry name="lfmetacarpal_visual">
-	  <mesh filename="package://sr_hand/model/meshes/lfmetacarpal.mesh" scale="0.001 0.001 0.001" />
-	</geometry>
-	<material name="Grey" />
+        <origin xyz="0 0 0" rpy="0 0 0" />
+        <geometry name="lfmetacarpal_visual">
+          <mesh filename="package://sr_hand/model/meshes/${mesh}" scale="0.001 0.001 0.001" />
+        </geometry>
+        <material name="Grey" />
       </visual>
       <collision>
-	<origin xyz="-0.015 0 0.015" rpy="0 0 0" />
-	<geometry name="lfmetacarpal_collision_geom">
-	  <box size="0.005 0.005 0.03" />
-	</geometry>
+          <origin xyz="${reflect*-0.015} 0 0.015" rpy="0 0 0" />
+        <geometry name="lfmetacarpal_collision_geom">
+          <box size="0.005 0.005 0.03" />
+        </geometry>
       </collision>
     </link>
@@ -47,54 +55,6 @@
       <parent link="${parent}"/>
       <child link="lfmetacarpal"/>
-      <origin xyz="-0.033 0 0.02071" rpy="0 0 0" />
-      <axis xyz="0.573576436 0 0.819152044" />
-      <limit lower="0" upper="0.69813170079773179" effort="10"
-      velocity="1.0" />
-      <dynamics damping="50.5"/>
-    </joint>
-    <xacro:lfmetacarpal_transmission />
-  </xacro:macro>
-  <!-- Left Handed -->
-  <xacro:macro name="lfmetacarpal_left" params="parent">
-    <link name="lfmetacarpal">
-      <inertial>
-	<origin xyz="0.033 0 0.02071" rpy="0 0 0" />
-	<mass value="0.075" />
-	<inertia  ixx="0.1" ixy="0.0"  ixz="0.0"  iyy="0.1"  iyz="0.0"
-	izz="0.1" />
-      </inertial>
-      <visual>
-	<origin xyz="0 0 0" rpy="0 0 0" />
-	<geometry name="lfmetacarpal_visual">
-	  <mesh filename="package://sr_hand/model/meshes/lfmetacarpal_left.mesh" scale="0.001 0.001 0.001" />
-	</geometry>
-	<material name="Grey" />
-      </visual>
-      <collision>
-	<origin xyz="0.015 0 0.015" rpy="0 0 0" />
-	<geometry name="lfmetacarpal_collision_geom">
-	  <box size="0.005 0.005 0.03" />
-	</geometry>
-      </collision>
-    </link>
-    <gazebo reference="lfmetacarpal">
-      <sensor:contact name="lfmetacarpal_contact_sensor">
-        <geom>lfmetacarpal_geom</geom>
-       <updateRate>100.0</updateRate>
-        <controller:gazebo_ros_bumper name="lfmetacarpal_gazebo_ros_bumper_controller" plugin="libgazebo_ros_bumper.so">
-          <alwaysOn>true</alwaysOn>
-          <updateRate>100.0</updateRate>
-          <frameName>lfmetacarpal</frameName>
-          <bumperTopicName>lfmetacarpal_bumper</bumperTopicName>
-          <interface:bumper name="lfmetacarpal_gazebo_ros_bumper_iface" />
-        </controller:gazebo_ros_bumper>
-      </sensor:contact>
-      <material>Gazebo/Grey</material>
-    </gazebo>
-    <joint name="LFJ5" type="revolute">
-      <parent link="${parent}"/>
-      <child link="lfmetacarpal"/>
-      <origin xyz="0.033 0 0.02071" rpy="0 0 0" />
-      <axis xyz="0.573576436 0 -0.819152044" />
+      <origin xyz="${reflect*-0.033} 0 0.02071" rpy="0 0 0" />
+      <axis xyz="0.573576436 0 ${reflect*0.819152044}" />
       <limit lower="0" upper="0.69813170079773179" effort="10"
       velocity="1.0" />

File: model/hand_urdf/finger/little_finger.urdf.xacro (robot description, xacro)
@@ -13,66 +13,16 @@
   <!-- Right Handed -->
   <xacro:macro name="little_finger" params="link_prefix joint_prefix parent">
-    <xacro:lfmetacarpal parent="${parent}">
-    </xacro:lfmetacarpal>
-    <link name="lfknuckle">
-      <inertial>
-        <origin xyz="0 0 0.06579" rpy="0 0 0" />
-        <mass value="0.008" />
-        <inertia ixx="0.1" ixy="0.0" ixz="0.0" iyy="0.1" iyz="0.0" izz="0.1" />
-      </inertial>
-      <visual>
-        <origin xyz="0 0 0" rpy="0 0 0" />
-        <geometry name="knuckle_visual">
-          <mesh filename="package://sr_hand/model/meshes/knuckle.mesh" scale="0.001 0.001 0.001" />
-        </geometry>
-        <material name="LightGrey" />
-      </visual>
-      <collision>
-        <origin xyz="0 0 0" rpy="0 0 0" />
-        <geometry name="knuckle_collision_geom">
-          <box size="0.005 0.005 0.005" />
-        </geometry>
-      </collision>
-    </link>
-    <gazebo reference="lfknuckle">
-      <sensor:contact name="lfknuckle_contact_sensor">
-        <geom>lfknuckle_geom</geom>
-        <updateRate>100.0</updateRate>
-        <controller:gazebo_ros_bumper name="lfknuckle_gazebo_ros_bumper_controller" plugin="libgazebo_ros_bumper.so">
-          <alwaysOn>true</alwaysOn>
-          <updateRate>100.0</updateRate>
-          <frameName>lfknuckle</frameName>
-          <bumperTopicName>lfknuckle_bumper</bumperTopicName>
-          <interface:bumper name="lfknuckle_gazebo_ros_bumper_iface" />
-        </controller:gazebo_ros_bumper>
-      </sensor:contact>
-      <material>PR2/Grey2</material>
-    </gazebo>
-    <joint name="LFJ4" type="revolute">
-      <parent link="lfmetacarpal" />
-      <child link="lfknuckle" />
-      <origin xyz="0 0 0.06579" rpy="0 0 0" />
-      <axis xyz="0 1 0" />
-      <limit lower="-0.43633231299858238" upper="0.43633231299858238" effort="10" velocity="1.0" />
-      <dynamics damping="50.5" />
-    </joint>
-    <transmission type="sr_mechanism_model/SimpleTransmission" name="lfknuckle_transmission">
-      <actuator name="LFJ4" />
-      <joint name="LFJ4" />
-      <mechanicalReduction>1</mechanicalReduction>
-      <motorTorqueConstant>1</motorTorqueConstant>
-      <pulsesPerRevolution>90000</pulsesPerRevolution>
-    </transmission>
-    <xacro:proximal link_prefix="${link_prefix}" joint_prefix="${joint_prefix}" parent="${link_prefix}knuckle">
-    </xacro:proximal>
-    <xacro:middle link_prefix="${link_prefix}" joint_prefix="${joint_prefix}" parent="${link_prefix}proximal">
-    </xacro:middle>
-    <xacro:distal link_prefix="${link_prefix}" joint_prefix="${joint_prefix}" parent="${link_prefix}middle">
-    </xacro:distal>
+    <xacro:lfmetacarpal parent="${parent}" />
+    <xacro:little_finger_common link_prefix="${link_prefix}" joint_prefix="${joint_prefix}" parent="${parent}" />
   </xacro:macro>
   <!-- Left Handed -->
   <xacro:macro name="little_finger_left" params="link_prefix joint_prefix parent">
-    <xacro:lfmetacarpal_left parent="${parent}">
-    </xacro:lfmetacarpal_left>
+    <xacro:lfmetacarpal_left parent="${parent}" />
+    <xacro:little_finger_common link_prefix="${link_prefix}" joint_prefix="${joint_prefix}" parent="${parent}" />
+  </xacro:macro>
+  <!-- Common bits for left handed and right handed little fingers. For use in
+  macros above to generate little_finger and little_finger_left.
+  DO NOT use out side of here ie treat as a private macro -->
+  <xacro:macro name="little_finger_common" params="link_prefix joint_prefix parent">
     <link name="lfknuckle">
       <inertial>
