Commit message: modified models to correct some small bugs

File: model/arm_urdf/upper_arm/shadowarm_upperarm.urdf.xacro (robot description, xacro)
@@ -29,5 +29,5 @@
       <parent link="${parent}"/>
       <child link="shadowarm_upperarm"/>
-      <origin xyz="0 -0.134 0.5405" rpy="0 -${M_PI} 0" />
+      <origin xyz="0 -0.134 0.5305" rpy="0 -${M_PI} 0" />
       <axis xyz="0 -1 0" />
       <limit lower="0" upper="${M_PI/2}" effort="10" velocity="1.0"/>

File: model/hand_urdf/finger/distal/distal.urdf.xacro (robot description, xacro)
@@ -23,7 +23,7 @@
       </visual>
       <collision>
-	<origin xyz="0 0 0.02" rpy="0 0 0" />
+	<origin xyz="0 0 0" rpy="0 0 0" />
 	<geometry name="distal_collision_geom">
-	  <box size="0.015 0.015 0.020" />
+	  <mesh filename="package://sr_hand/model/meshes/F1.mesh" scale="0.001 0.001 0.001" />
 	</geometry>
       </collision>

File: model/hand_urdf/finger/distal/distal_ellipsoid.urdf.xacro (robot description, xacro)
@@ -18,21 +18,14 @@
 	<origin xyz="0 0 0" rpy="0 0 0" />
 	<geometry name="distal_visual">
-      <mesh filename="package://sr_hand/model/meshes/distal_ellipsoid.mesh" scale="0.001 0.001 0.001" />
-    </geometry>
-      <material name="Grey" />
+	  <mesh filename="package://sr_hand/model/meshes/distal_ellipsoid.mesh" scale="0.001 0.001 0.001" />
+	</geometry>
+	<material name="Grey" />
       </visual>
-<!--      <visual>
+      <collision>
 	<origin xyz="0 0 0" rpy="0 0 0" />
-	<geometry name="nano17">
-      <mesh filename="package://sr_hand/model/meshes/nano17.mesh" scale="0.001 0.001 0.001" />
-      </geometry>
-     <material name="Grey" />
-      </visual>-->
-      <collision>
-		<origin xyz="0 0 0.02" rpy="0 0 0" />
-			<geometry name="distal_collision_geom">
-			  <box size="0.015 0.015 0.020" />
-			</geometry>
-	  </collision>
+	<geometry name="distal_collision_geom">
+	  <mesh filename="package://sr_hand/model/meshes/distal_ellipsoid.mesh" scale="0.001 0.001 0.001" />
+	</geometry>
+      </collision>
     </link>
     <gazebo reference="${link_prefix}distal">

File: model/hand_urdf/thumb/thdistal_ellipsoid.urdf.xacro (robot description, xacro)
@@ -25,7 +25,7 @@
       </visual>
       <collision>
-	<origin xyz="0 0 0.025" rpy="0 0 0 " />
+	<origin xyz="0 0.002 0.0025" rpy="0 0 0 " />
 	<geometry name="thmiddle_collision_geom">
-	  <box size="0.015 0.015 0.015" />
+	  <mesh filename="package://sr_hand/model/meshes/distal_ellipsoid.mesh" scale="0.001 0.001 0.001" />
 	</geometry>
       </collision>
