Commit message: lp:844934 working on ensuring the compatibility with electric

File: model/arm_urdf/base/shadowarm_base.urdf.xacro (robot description, xacro)
@@ -27,9 +27,4 @@
     <selfCollide>true</selfCollide>
   </gazebo>
-  <joint name="base_fix" type="fixed">
-    <parent link="world"/>
-    <child link="shadowarm_base"/>
-    <origin rpy="0 0 0" xyz="0 0 0"/>
-  </joint>
 </xacro:macro>
 </robot>

File: model/desk/desk.urdf.xacro (robot description, xacro)
@@ -23,4 +23,8 @@
   <gazebo reference="desk_pillar">
     <material>Gazebo/Green</material>
+    <mu1>1000.0</mu1>
+    <mu2>1000.0</mu2>
+    <kp>10000000.0</kp>
+    <kd>1.0</kd>
     <selfCollide>true</selfCollide>
   </gazebo>
@@ -47,5 +51,12 @@
   <gazebo reference="desk_support">
     <material>Gazebo/Green</material>
+    <mu1>1000.0</mu1>
+    <mu2>1000.0</mu2>
+    <kp>10000000.0</kp>
+    <kd>1.0</kd>
     <selfCollide>true</selfCollide>
+  </gazebo>
+  <gazebo>
+    <canonicalBody>desk_support</canonicalBody>
   </gazebo>
   <joint name="desk_joint" type="fixed">

File: model/robots/xacro/arm_and_hand_motor.urdf.xacro (robot description, xacro)
@@ -6,8 +6,13 @@
   <include filename="$(find sr_hand)/model/desk/desk.urdf.xacro" />
   <xacro:desk/>
-  <joint name="base_fix" type="fixed">
+  <joint name="arm_to_desk_fixed" type="fixed">
     <parent link="desk_pillar"/>
     <child link="shadowarm_base"/>
     <origin rpy="0 0 0" xyz="0 0 1.0"/>
+  </joint>
+  <joint name="base_fix" type="fixed">
+    <parent link="world"/>
+    <child link="desk_support"/>
+    <origin rpy="0 0 0" xyz="0 0 0"/>
   </joint>
   <xacro:sr_arm_motor>

Commit message: Arm meshes upgrade (simplified and corrected orientation) Adapted arm_urdf to rpy 0 0 0 since meshes are correctly oriented

File: model/arm_urdf/base/shadowarm_base.urdf.xacro (robot description, xacro)
@@ -10,5 +10,5 @@
     </inertial>
     <visual>
-      <origin xyz="0 0 0.005" rpy="${M_PI/2} 0 0"/>
+      <origin xyz="0 0 0.005" rpy="0 0 0"/>
       <geometry name="shadowarm_base_visual">
         <mesh filename="package://sr_hand/model/meshes/arm/arm_base.mesh" scale="0.001 0.001 0.001" />

File: model/arm_urdf/hand_support/shadowarm_handsupport_motor.urdf.xacro (robot description, xacro)
@@ -9,5 +9,5 @@
       </inertial>
       <visual>
-	<origin xyz="0 0 -0.04" rpy="${M_PI/2} 0 0"/>
+	<origin xyz="0 0 -0.04" rpy="0 0 0"/>
 	<geometry name="shadowarm_handsupport_visual">
 	  <mesh filename="package://sr_hand/model/meshes/arm/elbow_rotate_motor.mesh" scale="0.001 0.001 0.001" />

File: model/arm_urdf/lower_arm/shadowarm_lowerarm.urdf.xacro (robot description, xacro)
@@ -9,5 +9,5 @@
 	</inertial>
 	<visual>
-	  <origin xyz="0.03 0 0.036" rpy="${M_PI} ${0.5-M_PI/2} 0"/>
+	  <origin xyz="0.03 0 0.036" rpy="0 0 0"/>
 	  <geometry name="shadowarm_lowerarm_visual">
 	    <mesh filename="package://sr_hand/model/meshes/arm/elbow_flex.mesh" scale="0.001 0.001 0.001" />

File: model/arm_urdf/trunk/shadowarm_trunk.urdf.xacro (robot description, xacro)
@@ -9,5 +9,5 @@
 	</inertial>
 	<visual>
-	  <origin xyz="0 0 0.0165" rpy="${M_PI/2} ${M_PI} ${M_PI/2}" />
+	  <origin xyz="0 0 0.0165" rpy="0 0 0" />
 	  <geometry name="shadowarm_trunk_visual">
 	    <mesh filename="package://sr_hand/model/meshes/arm/arm_trunk.mesh" scale="0.001 0.001 0.001" />

File: model/arm_urdf/upper_arm/shadowarm_upperarm.urdf.xacro (robot description, xacro)
@@ -9,5 +9,5 @@
       </inertial>
       <visual>
-	<origin xyz="0 0.067 0" rpy="0 0 -${M_PI/2}" />
+	<origin xyz="0 0.067 0" rpy="0 0 0" />
 	<geometry name="shadowarm_upperarm_visual">
 	  <mesh filename="package://sr_hand/model/meshes/arm/upper_arm.mesh" scale="0.001 0.001 0.001" />

Commit message: Correct kinematics (arm and hand) Corrected collision boxes (no reflection, no offset) and added new tip links Moved to .dae meshes (did not include muscle and left stuff) Fixed vibrating issues in gazebo and retuned the controllers Corrected CAN compat to use generic name Improved friction of fingertips in gazebo Added a Kinect (model + attached to the arm) Added getJointState service Added joint_spline_trajectory controller for smoother arm movements Corrected trajectory message in joint_trajectory_controller to be compatible with new messages Removed deprecated sendupdate calls in joint_trajectory_controller Corrected urdf description call in launch files (now using sa and sh instead of arm or hand) Added new launch files (stand_alone versions)

File: model/arm_urdf/base/shadowarm_base.urdf.xacro (robot description, xacro)
@@ -10,7 +10,7 @@
     </inertial>
     <visual>
-      <origin xyz="0 0 0.005" rpy="0 0 0"/>
+      <origin xyz="0 0 0" rpy="0 0 0"/>
       <geometry name="shadowarm_base_visual">
-        <mesh filename="package://sr_hand/model/meshes/arm/arm_base.mesh" scale="0.001 0.001 0.001" />
+        <mesh filename="package://sr_hand/model/meshes/arm/arm_base.dae" scale="0.001 0.001 0.001" />
       </geometry>
       <material name="LightGrey" />

File: model/arm_urdf/hand_support/shadowarm_handsupport_motor.urdf.xacro (robot description, xacro)
@@ -11,10 +11,10 @@
 	<origin xyz="0 0 -0.04" rpy="0 0 0"/>
 	<geometry name="shadowarm_handsupport_visual">
-	  <mesh filename="package://sr_hand/model/meshes/arm/elbow_rotate_motor.mesh" scale="0.001 0.001 0.001" />
+	  <mesh filename="package://sr_hand/model/meshes/arm/elbow_rotate_motor.dae" scale="0.001 0.001 0.001" />
 	</geometry>
 	<material name="LightGrey" />
       </visual>
       <collision>
-	<origin xyz="0 0 0" rpy="0 0 0"/>
+	<origin xyz="0 0 -0.005" rpy="0 0 0"/>
 	<geometry name="shadowarm_handsupport_collision">
 	  <cylinder radius="0.06" length="0.001"/>
@@ -29,5 +29,5 @@
       <parent link="${parent}"/>
       <child link="shadowarm_handsupport_motor"/>
-      <origin xyz="0.08 0 0.131" rpy="0 0 0" />
+      <origin xyz="0.08 0 0.125" rpy="0.0 0 0" />
       <axis xyz="0 0 -1" />
       <limit lower="-${M_PI/2}" upper="${M_PI/2}"

File: model/arm_urdf/lower_arm/shadowarm_lowerarm.urdf.xacro (robot description, xacro)
@@ -4,5 +4,5 @@
     <link name="shadowarm_lowerarm">
 	<inertial>
-	  <origin xyz="0.08 0 0.0655" rpy="0 0 0" />
+	  <origin xyz="0.08 0 0.0625" rpy="0 0 0" />
 	  <mass value="1.7" />
 	  <inertia  ixx="1.0" ixy="0.0"  ixz="0.0"  iyy="0.0"  iyz="0.0"  izz="0.0" />
@@ -11,12 +11,12 @@
 	  <origin xyz="0.03 0 0.036" rpy="0 0 0"/>
 	  <geometry name="shadowarm_lowerarm_visual">
-	    <mesh filename="package://sr_hand/model/meshes/arm/elbow_flex.mesh" scale="0.001 0.001 0.001" />
+	    <mesh filename="package://sr_hand/model/meshes/arm/elbow_flex.dae" scale="0.001 0.001 0.001" />
 	  </geometry>
 	  <material name="Grey" />
 	</visual>
 	<collision>
-	  <origin xyz="0.08 0 0.0655" rpy="0 0 0"/>
+	  <origin xyz="0.08 0 0.0625" rpy="0 0 0"/>
 	  <geometry name="shadowarm_lowerarm_collision">
-	    <box size="0.03 0.03 0.131"/>
+	    <box size="0.03 0.03 0.10"/>
 	  </geometry>
 	</collision>
@@ -31,5 +31,5 @@
       <origin xyz="0 0 0.369" rpy="0 0 0" />
       <axis xyz="0 -1 0" />
-      <limit lower="0" upper="2.09439510239"
+      <limit lower="0.52" upper="2.09439510239"
       effort="10" velocity="1.0"/>
       <dynamics damping="50.5"/>

File: model/arm_urdf/trunk/shadowarm_trunk.urdf.xacro (robot description, xacro)
@@ -4,19 +4,19 @@
     <link name="shadowarm_trunk">
 	<inertial>
-	  <origin xyz="0 0 0.27025" rpy="0 0 0" />
+	  <origin xyz="0 0 0.26525" rpy="0 0 0" />
 	  <mass value="10" />
 	  <inertia  ixx="1.47" ixy="0.0"  ixz="0.0"  iyy="1.47"  iyz="0.0"  izz="2.4" />
 	</inertial>
 	<visual>
-	  <origin xyz="0 0 0.0165" rpy="0 0 0" />
+	  <origin xyz="0 0 0.005" rpy="0 0 0" />
 	  <geometry name="shadowarm_trunk_visual">
-	    <mesh filename="package://sr_hand/model/meshes/arm/arm_trunk.mesh" scale="0.001 0.001 0.001" />
+	    <mesh filename="package://sr_hand/model/meshes/arm/arm_trunk.dae" scale="0.001 0.001 0.001" />
 	  </geometry>
 	  <material name="Grey" />
 	</visual>
 	<collision>
-	  <origin xyz="0 0 0.27025" rpy="0 0 0"/>
+	  <origin xyz="0 0 0.26525" rpy="0 0 0"/>
 	  <geometry name="shadowarm_trunk_collision">
-	    <box size="0.03 0.03 0.5405"/>
+	    <box size="0.03 0.03 0.52"/>
 	  </geometry>
 	</collision>
@@ -29,5 +29,5 @@
       <parent link="${parent}"/>
       <child link="shadowarm_trunk"/>
-      <origin xyz="0 0 0.01" rpy="0 0 0" />
+      <origin xyz="0 0 0.01" rpy="0.0 0.0 0.0" />
       <axis xyz="0 0 1" />
       <limit lower="-${M_PI/4}" upper="${M_PI/2}"

File: model/arm_urdf/upper_arm/shadowarm_upperarm.urdf.xacro (robot description, xacro)
@@ -4,5 +4,5 @@
     <link name="shadowarm_upperarm">
       <inertial>
-	<origin xyz="0 -0.067 -0.1845" rpy="0 0 0" />
+	<origin xyz="0 0 0.1845" rpy="0 0 0" />
 	<mass value="2" />
 	<inertia  ixx="0.5" ixy="0.0"  ixz="0.0"  iyy="0.5"  iyz="0.0"  izz="0.1" />
@@ -11,5 +11,5 @@
 	<origin xyz="0 0.067 0" rpy="0 0 0" />
 	<geometry name="shadowarm_upperarm_visual">
-	  <mesh filename="package://sr_hand/model/meshes/arm/upper_arm.mesh" scale="0.001 0.001 0.001" />
+	  <mesh filename="package://sr_hand/model/meshes/arm/upper_arm.dae" scale="0.001 0.001 0.001" />
 	</geometry>
 	<material name="Grey" />
@@ -29,5 +29,5 @@
       <parent link="${parent}"/>
       <child link="shadowarm_upperarm"/>
-      <origin xyz="0 -0.134 0.5305" rpy="0 -${M_PI} 0" />
+      <origin xyz="0 -0.134 0.5305" rpy="0 -${M_PI} 0.0" /> <!-- yaw=-0.026 -->
       <axis xyz="0 -1 0" />
       <limit lower="0" upper="${M_PI/2}" effort="10" velocity="1.0"/>

File: model/desk/desk.urdf.xacro (robot description, xacro)
@@ -4,18 +4,18 @@
     <inertial>
       <origin xyz="0 0 0.5"/>
-      <mass value="100.0"/>
-      <inertia ixx="1.0" ixy="0.0" ixz="0.0" iyy="0.0" iyz="0.0" izz="0.0"/>
+      <mass value="1000.0"/>
+      <inertia ixx="1.0" ixy="0.0" ixz="0.0" iyy="1.0" iyz="0.0" izz="1.0"/>
     </inertial>
     <visual>
-      <origin rpy="0 0 0" xyz="0 0 0.5"/>
+      <origin rpy="0 0 0" xyz="0 0 0.51"/>
       <geometry name="desk_visual">
-        <cylinder length="1.0" radius="0.1"/>
+        <cylinder length="0.98" radius="0.1"/>
       </geometry>
       <material name="Green"/>
     </visual>
     <collision>
-      <origin rpy="0 0 0" xyz="0 0 0.5"/>
+      <origin rpy="0 0 0" xyz="0 0 0.51"/>
       <geometry name="desk_collision">
-        <cylinder length="1.0" radius="0.1"/>
+        <cylinder length=".98" radius="0.1"/>
       </geometry>
     </collision>
@@ -31,7 +31,7 @@
   <link name="desk_support">
     <inertial>
-      <origin xyz="0 0 0.01"/>
+      <origin xyz="0 0 0"/>
       <mass value="1000.0"/>
-      <inertia ixx="1.0" ixy="0.0" ixz="0.0" iyy="0.0" iyz="0.0" izz="0.0"/>
+      <inertia ixx="1.0" ixy="0.0" ixz="0.0" iyy="1.0" iyz="0.0" izz="1.0"/>
     </inertial>
     <visual>
@@ -63,5 +63,5 @@
     <parent link="desk_support"/>
     <child link="desk_pillar"/>
-    <origin rpy="0 0 0" xyz="0 0 0.01"/>
+    <origin rpy="0 0 0" xyz="0 0 0.02"/>
   </joint>
   </xacro:macro>

File: model/hand_urdf/finger/distal/distal.urdf.xacro (robot description, xacro)
@@ -11,5 +11,5 @@
       <inertial>
 	<mass value="0.010" />
-	<origin xyz="0 0 0.025" />
+	<origin xyz="0 0 0.013" />
 	<inertia  ixx="0.1" ixy="0.0"  ixz="0.0"  iyy="0.1"  iyz="0.0"
 	izz="0.0" />
@@ -25,5 +25,5 @@
 	<origin xyz="0 0 0" rpy="0 0 0" />
 	<geometry name="distal_collision_geom">
-	  <mesh filename="package://sr_hand/model/meshes/F1.mesh" scale="0.001 0.001 0.001" />
+	 <mesh filename="package://sr_hand/model/meshes/F1.dae" scale="0.001 0.001 0.001" />
 	</geometry>
       </collision>
@@ -41,5 +41,10 @@
         </controller:gazebo_ros_bumper>
       </sensor:contact>
+      <mu1 value="500.0" />
+      <mu2 value="500.0" />
+      <kp  value="10000000.0" />
+      <kd  value="1.0" />
       <material>Gazebo/Grey</material>
+      <selfCollide>false</selfCollide>
     </gazebo>
     <joint name="${joint_prefix}J1" type="revolute">
@@ -52,4 +57,15 @@
       <dynamics damping="50.5"/>
     </joint>
+    <link name="${link_prefix}tip">
+			<inertial>
+				<mass value="0.001" />
+				<inertia  ixx="0.0" ixy="0.0"  ixz="0.0"  iyy="0.0"  iyz="0.0" izz="0.0" />
+  		</inertial>
+    </link>
+    <joint name="${joint_prefix}tip" type="fixed">
+      <parent link="${link_prefix}distal"/>
+      <child link="${link_prefix}tip"/>
+      <origin xyz="0 0 0.026" rpy="0 0 0" />
+    </joint>
 <!--
     <xacro:distal_transmission />

File: model/hand_urdf/finger/distal/distal_biotac.urdf.xacro (robot description, xacro)
@@ -11,5 +11,5 @@
       <inertial>
 	<mass value="0.010" />
-	<origin xyz="0 0 0.025" />
+	<origin xyz="0 0 0.013" />
 	<inertia  ixx="0.1" ixy="0.0"  ixz="0.0"  iyy="0.1"  iyz="0.0"
 	izz="0.0" />

File: model/hand_urdf/finger/distal/distal_ellipsoid.urdf.xacro (robot description, xacro)
@@ -11,5 +11,5 @@
       <inertial>
 	<mass value="0.010" />
-	<origin xyz="0 0 0.025" />
+	<origin xyz="0 0 0.013" />
 	<inertia  ixx="0.1" ixy="0.0"  ixz="0.0"  iyy="0.1"  iyz="0.0"
 	izz="0.0" />
@@ -18,13 +18,20 @@
 	<origin xyz="0 0 0" rpy="0 0 0" />
 	<geometry name="distal_visual">
-	  <mesh filename="package://sr_hand/model/meshes/distal_ellipsoid.mesh" scale="0.001 0.001 0.001" />
-	</geometry>
-	<material name="Grey" />
+      <mesh filename="package://sr_hand/model/meshes/distal_ellipsoid.dae" scale="0.001 0.001 0.001" />
+    </geometry>
+      <material name="Grey" />
       </visual>
+<!--      <visual>
+	<origin xyz="0 0 0" rpy="0 0 0" />
+	<geometry name="nano17">
+      <mesh filename="package://sr_hand/model/meshes/nano17.dae" scale="0.001 0.001 0.001" />
+      </geometry>
+     <material name="Grey" />
+      </visual>-->
       <collision>
-	<origin xyz="0 0 0" rpy="0 0 0" />
-	<geometry name="distal_collision_geom">
-	  <mesh filename="package://sr_hand/model/meshes/distal_ellipsoid.mesh" scale="0.001 0.001 0.001" />
-	</geometry>
+        <origin xyz="0 0 0" rpy="0 0 0" />
+        <geometry name="distal_collision_geom">
+          <mesh filename="package://sr_hand/model/meshes/distal_ellipsoid.dae" scale="0.001 0.001 0.001" />
+        </geometry>
       </collision>
     </link>
@@ -41,5 +48,10 @@
         </controller:gazebo_ros_bumper>
       </sensor:contact>
-      <material>Gazebo/Grey</material>
+     <mu1 value="500.0" />
+      <mu2 value="500.0" />
+      <kp  value="10000000.0" />
+      <kd  value="1.0" />
+     <material>Gazebo/Grey</material>
+	 <selfCollide>false</selfCollide>
     </gazebo>
     <joint name="${joint_prefix}J1" type="revolute">
@@ -52,4 +64,15 @@
       <dynamics damping="50.5"/>
     </joint>
+   <link name="${link_prefix}tip">
+			<inertial>
+				<mass value="0.001" />
+				<inertia  ixx="0.0" ixy="0.0"  ixz="0.0"  iyy="0.0"  iyz="0.0" izz="0.0" />
+  		</inertial>
+    </link>
+    <joint name="${joint_prefix}tip" type="fixed">
+      <parent link="${link_prefix}distal"/>
+      <child link="${link_prefix}tip"/>
+      <origin xyz="0 0 0.026" rpy="0 0 0" />
+    </joint>
 <!--
     <xacro:distal_transmission />

File: model/hand_urdf/finger/knuckle/knuckle.urdf.xacro (robot description, xacro)
@@ -10,6 +10,6 @@
     <link name="${link_prefix}knuckle">
       <inertial>
-	<!--<origin xyz="0.011 0 0.099" rpy="0 0 0" />-->
-	<insert_block name="origin" />
+	<origin xyz="0 0 0" rpy="0 0 0" />
+	<!--<insert_block name="origin" /> -->
 	<mass value="0.008" />
 	<inertia  ixx="0.0" ixy="0.0"  ixz="0.0"  iyy="0.1"  iyz="0.0"
@@ -19,5 +19,5 @@
 	<origin xyz="0 0 0.0005" rpy="0 0 0" />
 	<geometry name="knuckle_visual">
-      <mesh filename="package://sr_hand/model/meshes/knuckle.mesh" scale="0.001 0.001 0.001" />
+      <mesh filename="package://sr_hand/model/meshes/knuckle.dae" scale="0.001 0.001 0.001" />
       </geometry>
       <material name="LightGrey" />

File: model/hand_urdf/finger/lfmetacarpal/lfmetacarpal.urdf.xacro (robot description, xacro)
@@ -9,5 +9,5 @@
   <!-- Right Handed -->
   <xacro:macro name="lfmetacarpal" params="parent">
-      <xacro:lfmetacarpal_base parent="${parent}" reflect="1" mesh="lfmetacarpal.mesh" />
+      <xacro:lfmetacarpal_base parent="${parent}" reflect="1" mesh="lfmetacarpal.dae" />
   </xacro:macro>
   <!-- Left Handed -->
@@ -20,5 +20,5 @@
     <link name="lfmetacarpal">
       <inertial>
-        <origin xyz="${reflect*-0.033} 0 0.02071" rpy="0 0 0" />
+        <origin xyz="0 0 0.04" rpy="0 0 0" />
 	    <mass value="0.075" />
 	    <inertia  ixx="0.1" ixy="0.0"  ixz="0.0"  iyy="0.1"  iyz="0.0" izz="0.1" />
@@ -32,7 +32,7 @@
       </visual>
       <collision>
-          <origin xyz="${reflect*-0.015} 0 0.015" rpy="0 0 0" />
+          <origin xyz="0 0 0.04" rpy="0 0 0" />
         <geometry name="lfmetacarpal_collision_geom">
-          <box size="0.005 0.005 0.03" />
+          <box size="0.008 0.008 0.03" />
         </geometry>
       </collision>

File: model/hand_urdf/finger/little_finger.urdf.xacro (robot description, xacro)
@@ -27,5 +27,5 @@
     <link name="lfknuckle">
       <inertial>
-        <origin xyz="0 0 0.06579" rpy="0 0 0" />
+        <origin xyz="0 0 0" rpy="0 0 0" />
         <mass value="0.008" />
         <inertia ixx="0.1" ixy="0.0" ixz="0.0" iyy="0.1" iyz="0.0" izz="0.1" />
@@ -34,5 +34,5 @@
         <origin xyz="0 0 0" rpy="0 0 0" />
         <geometry name="knuckle_visual">
-          <mesh filename="package://sr_hand/model/meshes/knuckle.mesh" scale="0.001 0.001 0.001" />
+          <mesh filename="package://sr_hand/model/meshes/knuckle.dae" scale="0.001 0.001 0.001" />
         </geometry>
         <material name="LightGrey" />

File: model/hand_urdf/finger/little_finger_biotac.urdf.xacro (robot description, xacro)
@@ -27,5 +27,5 @@
     <link name="lfknuckle">
       <inertial>
-        <origin xyz="0 0 0.06579" rpy="0 0 0" />
+        <origin xyz="0 0 0.0" rpy="0 0 0" />
         <mass value="0.008" />
         <inertia ixx="0.1" ixy="0.0" ixz="0.0" iyy="0.1" iyz="0.0" izz="0.1" />
@@ -34,5 +34,5 @@
         <origin xyz="0 0 0" rpy="0 0 0" />
         <geometry name="knuckle_visual">
-          <mesh filename="package://sr_hand/model/meshes/knuckle.mesh" scale="0.001 0.001 0.001" />
+          <mesh filename="package://sr_hand/model/meshes/knuckle.dae" scale="0.001 0.001 0.001" />
         </geometry>
         <material name="LightGrey" />

File: model/hand_urdf/finger/little_finger_ellipsoid.urdf.xacro (robot description, xacro)
@@ -24,5 +24,5 @@
 	<origin xyz="0 0 0" rpy="0 0 0" />
 	<geometry name="knuckle_visual">
-      <mesh filename="package://sr_hand/model/meshes/knuckle.mesh" scale="0.001 0.001 0.001" />
+      <mesh filename="package://sr_hand/model/meshes/knuckle.dae" scale="0.001 0.001 0.001" />
       </geometry>
       <material name="LightGrey" />

File: model/hand_urdf/finger/middle/middle.urdf.xacro (robot description, xacro)
@@ -10,5 +10,5 @@
     <link name="${link_prefix}middle">
       <inertial>
-	<origin xyz="0 0 0.045" rpy="0 0 0" />
+	<origin xyz="0 0 0.0125" rpy="0 0 0" />
 	<mass value="0.012" />
 	<inertia  ixx="0.1" ixy="0.0"  ixz="0.0"  iyy="0.1"  iyz="0.0"
@@ -18,5 +18,5 @@
 	<origin xyz="0 0 0" rpy="0 0 0" />
 	<geometry name="middle_visual">
-      <mesh filename="package://sr_hand/model/meshes/F2.mesh" scale="0.001 0.001 0.001" />
+      <mesh filename="package://sr_hand/model/meshes/F2.dae" scale="0.001 0.001 0.001" />
       </geometry>
       <material name="Grey" />
@@ -25,5 +25,5 @@
 	<origin xyz="0 0 0.0125" rpy="0 0 0" />
 	<geometry name="middle_collision_geom">
-	  <box size="0.005 0.005 0.010" />
+	  <box size="0.008 0.008 0.015" />
 	</geometry>
       </collision>

File: model/hand_urdf/finger/proximal/proximal.urdf.xacro (robot description, xacro)
@@ -11,5 +11,5 @@
       <inertial>
 	<mass value="0.014" />
-	<origin xyz="0 0 0" />
+	<origin xyz="0 0 0.0225" />
 	<inertia  ixx="0.1" ixy="0.0"  ixz="0.0"  iyy="0.1"  iyz="0.0"
 	izz="0.0" />
@@ -18,12 +18,12 @@
 	<origin xyz="0 0 0" rpy="0 0 0" />
 	<geometry name="proximal_visual">
-      <mesh filename="package://sr_hand/model/meshes/F3.mesh" scale="0.001 0.001 0.001" />
+      <mesh filename="package://sr_hand/model/meshes/F3.dae" scale="0.001 0.001 0.001" />
       </geometry>
       <material name="Grey" />
       </visual>
       <collision>
-	<origin xyz="0 0 0.0225" rpy="0 0 0 " />
+	<origin xyz="0 0 0.025" rpy="0 0 0 " />
 	<geometry name="proximal_collision_geom">
-	  <box size="0.005 0.005 0.04" />
+	  <box size="0.008 0.008 0.04" />
 	</geometry>
       </collision>

File: model/hand_urdf/forearm/forearm_motor.urdf.xacro (robot description, xacro)
@@ -4,5 +4,5 @@
     <link name="forearm_motor">
       <inertial>
-	<origin xyz="0 0 0" />
+	<origin xyz="0 0 0.09" rpy="0 0 0"/>
 	<mass value="3.0" />
 	<inertia  ixx="1.0" ixy="0.0"  ixz="0.0"  iyy="1.0"  iyz="0.0"  izz="1.0" />
@@ -11,5 +11,5 @@
 	<origin xyz="0 0 0" rpy="0 0 0" />
 	<geometry name="shadow_forearm_geom">
-	  <mesh filename="package://sr_hand/model/meshes/forearm.mesh" scale="0.001 0.001 0.001"/>
+	  <mesh filename="package://sr_hand/model/meshes/forearm.dae" scale="0.001 0.001 0.001"/>
 	</geometry>
 	<material name="Grey" />

File: model/hand_urdf/forearm/forearm_muscle.urdf.xacro (robot description, xacro)
@@ -4,5 +4,5 @@
     <link name="forearm_muscle">
       <inertial>
-	<origin xyz="0 0 0" />
+	<origin xyz="0 0 0.175" />
 	<mass value="3.0" />
 	<inertia  ixx="0.00735" ixy="0.0"  ixz="0.0"  iyy="0.00735"  iyz="0.0"  izz="0.0343" />

File: model/hand_urdf/palm/palm.urdf.xacro (robot description, xacro)
@@ -9,5 +9,5 @@
   <!-- Right Hand -->
   <xacro:macro name="palm" params="parent">
-    <xacro:palm_base parent="${parent}" mesh="palm.mesh" />
+    <xacro:palm_base parent="${parent}" mesh="palm.dae" />
   </xacro:macro>
   <!-- Left Hand -->
@@ -20,5 +20,5 @@
     <link name="palm" >
       <inertial>
-	<origin xyz="0 0 0.247" rpy="0 0 0" />
+	<origin xyz="0 0 0.035" rpy="0 0 0" />
 	<mass value="0.3" />
 	<inertia  ixx="0.5" ixy="0.0"  ixz="0.0"  iyy="0.5"  iyz="0.0"	izz="0.3" />

File: model/hand_urdf/thumb/thbase.urdf.xacro (robot description, xacro)
@@ -21,5 +21,5 @@
       <inertial>
 	<mass value="0.010" />
-    <origin xyz="${reflect*0.034} 0.0085 0.029" rpy="0 0 0"/>
+	  <origin xyz="0 0 0" rpy="0 0 0"/>
 	<inertia  ixx="0.0" ixy="0.0"  ixz="0.0"  iyy="0.0"  iyz="0.0"
 	izz="0.1" />
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