Commit message: Extracted and adapted modifications needed to shadow stack from the manip-electric version to be compatible with sr-manipulation electric and to run in real. Works without manipulation stack also, but requires some testing of all the launch files. New dae meshes are currently with wrong colors but are working.

File: model/hand_urdf/finger/distal/distal_ellipsoid.urdf.xacro (robot description, xacro)
@@ -1,5 +1,5 @@
 <robot xmlns:xacro="http://ros.org/wiki/xacro"
-	xmlns:sensor="http://playerstage.sourceforge.net/gazebo/xmlschema/#sensor"
-	xmlns:controller="http://playerstage.sourceforge.net/gazebo/xmlschema/#controller"
+       xmlns:sensor="http://playerstage.sourceforge.net/gazebo/xmlschema/#sensor"
+       xmlns:controller="http://playerstage.sourceforge.net/gazebo/xmlschema/#controller"
        xmlns:joint="http://playerstage.sourceforge.net/gazebo/xmlschema/#slider"
        xmlns:interface="http://playerstage.sourceforge.net/gazebo/xmlschema/#interface"
@@ -13,20 +13,20 @@
 	<origin xyz="0 0 0.013" />
 	<inertia  ixx="0.1" ixy="0.0"  ixz="0.0"  iyy="0.1"  iyz="0.0"
-	izz="0.0" />
+		  izz="0.0" />
       </inertial>
       <visual>
 	<origin xyz="0 0 0" rpy="0 0 0" />
 	<geometry name="distal_visual">
-      <mesh filename="package://sr_hand/model/meshes/distal_ellipsoid.dae" scale="0.001 0.001 0.001" />
-    </geometry>
-      <material name="Grey" />
+	  <mesh filename="package://sr_hand/model/meshes/distal_ellipsoid.dae" scale="0.001 0.001 0.001" />
+	</geometry>
+	<material name="Grey" />
       </visual>
-<!--      <visual>
-	<origin xyz="0 0 0" rpy="0 0 0" />
-	<geometry name="nano17">
-      <mesh filename="package://sr_hand/model/meshes/nano17.dae" scale="0.001 0.001 0.001" />
-      </geometry>
-     <material name="Grey" />
-      </visual>-->
+      <!--      <visual>
+	   <origin xyz="0 0 0" rpy="0 0 0" />
+	   <geometry name="nano17">
+	   <mesh filename="package://sr_hand/model/meshes/nano17.dae" scale="0.001 0.001 0.001" />
+	   </geometry>
+	   <material name="Grey" />
+	   </visual>-->
       <collision>
         <origin xyz="0 0 0" rpy="0 0 0" />
@@ -48,10 +48,10 @@
         </controller:gazebo_ros_bumper>
       </sensor:contact>
-     <mu1 value="500.0" />
+      <mu1 value="500.0" />
       <mu2 value="500.0" />
       <kp  value="10000000.0" />
       <kd  value="1.0" />
-     <material>Gazebo/Grey</material>
-	 <selfCollide>false</selfCollide>
+      <material>Gazebo/Grey</material>
+      <selfCollide>false</selfCollide>
     </gazebo>
     <joint name="${joint_prefix}J1" type="revolute">
@@ -61,12 +61,12 @@
       <axis xyz="1 0 0" />
       <limit lower="0" upper="${M_PI/2}" effort="10"
-      velocity="1.0" />
+	     velocity="1.0" />
       <dynamics damping="50.5"/>
     </joint>
-   <link name="${link_prefix}tip">
-			<inertial>
-				<mass value="0.001" />
-				<inertia  ixx="0.0" ixy="0.0"  ixz="0.0"  iyy="0.0"  iyz="0.0" izz="0.0" />
-  		</inertial>
+    <link name="${link_prefix}tip">
+      <inertial>
+	<mass value="0.001" />
+	<inertia  ixx="0.0" ixy="0.0"  ixz="0.0"  iyy="0.0"  iyz="0.0" izz="0.0" />
+      </inertial>
     </link>
     <joint name="${joint_prefix}tip" type="fixed">
@@ -75,7 +75,7 @@
       <origin xyz="0 0 0.026" rpy="0 0 0" />
     </joint>
-<!--
-    <xacro:distal_transmission />
--->
+    <!--
+	<xacro:distal_transmission />
+    -->
   </xacro:macro>
 </robot>

File: model/hand_urdf/thumb/thdistal.urdf.xacro (robot description, xacro)
@@ -13,12 +13,12 @@
 	<origin xyz="0 0 0.01375" rpy="0 0 0"/>
 	<inertia  ixx="0.1" ixy="0.0"  ixz="0.0"  iyy="0.1"  iyz="0.0"
-	izz="0.1" />
+		  izz="0.1" />
       </inertial>
       <visual>
 	<origin xyz="0 0 0" rpy="0 0 0" />
 	<geometry name="thdistal_visual">
-	<mesh filename="package://sr_hand/model/meshes/TH1_z.dae" scale="0.001 0.001 0.001" />
-      </geometry>
-      <material name="shadow_thmiddle_material">
+	  <mesh filename="package://sr_hand/model/meshes/TH1_z.dae" scale="0.001 0.001 0.001" />
+	</geometry>
+	<material name="shadow_thmiddle_material">
 	  <color rgba="0.2 0.2 0.2 1.0"/>
 	</material>
@@ -27,6 +27,6 @@
 	<origin xyz="0 0 0" rpy="0 0 0 " />
 	<geometry name="thmiddle_collision_geom">
-    	<mesh filename="package://sr_hand/model/meshes/TH1_z.dae" scale="0.001 0.001 0.001" />
-<!--	  <box size="0.015 0.015 0.015" /> -->
+	  <mesh filename="package://sr_hand/model/meshes/TH1_z.dae" scale="0.001 0.001 0.001" />
+	  <!--	  <box size="0.015 0.015 0.015" /> -->
 	</geometry>
       </collision>
@@ -35,5 +35,5 @@
       <sensor:contact name="thdistal_contact_sensor">
         <geom>thdistal_geom</geom>
-       <updateRate>100.0</updateRate>
+	<updateRate>100.0</updateRate>
         <controller:gazebo_ros_bumper name="thdistal_gazebo_ros_bumper_controller" plugin="libgazebo_ros_bumper.so">
           <alwaysOn>true</alwaysOn>
@@ -57,12 +57,12 @@
       <axis xyz="1 0 0" />
       <limit lower="0" upper="1.571" effort="10"
-      velocity="1.0" />
+	     velocity="1.0" />
       <dynamics damping="50.5"/>
     </joint>
     <link name="thtip">
-			<inertial>
-				<mass value="0.001" />
-				<inertia  ixx="0.0" ixy="0.0"  ixz="0.0"  iyy="0.0"  iyz="0.0" izz="0.0" />
-  		</inertial>
+      <inertial>
+	<mass value="0.001" />
+	<inertia  ixx="0.0" ixy="0.0"  ixz="0.0"  iyy="0.0"  iyz="0.0" izz="0.0" />
+      </inertial>
     </link>
     <joint name="thtip" type="fixed">

File: model/hand_urdf/thumb/thdistal_ellipsoid.urdf.xacro (robot description, xacro)
@@ -13,12 +13,12 @@
 	<origin xyz="0 0 0.01375" rpy="0 0 0"/>
 	<inertia  ixx="0.1" ixy="0.0"  ixz="0.0"  iyy="0.1"  iyz="0.0"
-	izz="0.1" />
+		  izz="0.1" />
       </inertial>
       <visual>
 	<origin xyz="0 0.002 0.0025" rpy="0 0 0" />
 	<geometry name="thdistal_visual">
-	<mesh filename="package://sr_hand/model/meshes/distal_ellipsoid.dae" scale="0.001 0.001 0.001" />
-      </geometry>
-      <material name="shadow_thmiddle_material">
+	  <mesh filename="package://sr_hand/model/meshes/distal_ellipsoid.dae" scale="0.001 0.001 0.001" />
+	</geometry>
+	<material name="shadow_thmiddle_material">
 	  <color rgba="0.2 0.2 0.2 1.0"/>
 	</material>
@@ -27,5 +27,5 @@
 	<origin xyz="0 0.002 0.0025" rpy="0 0 0 " />
 	<geometry name="thmiddle_collision_geom">
-	 <mesh filename="package://sr_hand/model/meshes/distal_ellipsoid.dae" scale="0.001 0.001 0.001" />
+	  <mesh filename="package://sr_hand/model/meshes/distal_ellipsoid.dae" scale="0.001 0.001 0.001" />
 	</geometry>
       </collision>
@@ -34,5 +34,5 @@
       <sensor:contact name="thdistal_contact_sensor">
         <geom>thdistal_geom</geom>
-       <updateRate>100.0</updateRate>
+	<updateRate>100.0</updateRate>
         <controller:gazebo_ros_bumper name="thdistal_gazebo_ros_bumper_controller" plugin="libgazebo_ros_bumper.so">
           <alwaysOn>true</alwaysOn>
@@ -56,12 +56,12 @@
       <axis xyz="1 0 0" />
       <limit lower="0" upper="1.571" effort="10"
-      velocity="1.0" />
+	     velocity="1.0" />
       <dynamics damping="50.5"/>
     </joint>
     <link name="thtip">
-			<inertial>
-				<mass value="0.001" />
-				<inertia  ixx="0.0" ixy="0.0"  ixz="0.0"  iyy="0.0"  iyz="0.0" izz="0.0" />
-  		</inertial>
+      <inertial>
+	<mass value="0.001" />
+	<inertia  ixx="0.0" ixy="0.0"  ixz="0.0"  iyy="0.0"  iyz="0.0" izz="0.0" />
+      </inertial>
     </link>
     <joint name="thtip" type="fixed">
