Commit message: Corrected colors and wrong texture on dae objects Corrected distal.urdf.xacro to use .dae

File: model/hand_urdf/finger/distal/distal.urdf.xacro (robot description, xacro)
@@ -18,5 +18,5 @@
 	<origin xyz="0 0 0" rpy="0 0 0" />
 	<geometry name="distal_visual">
-      <mesh filename="package://sr_hand/model/meshes/F1.mesh" scale="0.001 0.001 0.001" />
+      <mesh filename="package://sr_hand/model/meshes/F1.dae" scale="0.001 0.001 0.001" />
       </geometry>
       <material name="Grey" />
