Commit message: New versions of Hand and Arm finders

File: sr_utilities/test/urdf/no_hand_description.urdf (robot description, URDF)
Before this commit: robot no_hand_robot, 2 links, 1 joints
Links:
- removed link first_link
- added link la_first_link; visual cylinder length=1.0 radius=0.1
Joints:
- removed joint base_to_first_link
- added joint la_first_joint: type continuous, parent base_link, child la_first_link
